File: lab02/lab02.kicad_sch (KiCad schematic)
At the start: 0 parts

Commit message: main v0
Parts:
- added D2, D3, D4: GREEN LED, LED_SMD:LED_0603_1608Metric_Pad1.05x0.95mm_HandSolder, symbol Device:LED
- added R2, R3, R4: 56R, symbol Device:R_Small
- added R5, R6, R7: 100R, symbol Device:R_Small
- added SW1, SW2, SW3: SW_Push, symbol Switch:SW_Push
- added U2: ESP32-WROOM-32, RF_Module:ESP32-WROOM-32, symbol RF_Module:ESP32-WROOM-32
Connections:
- new net: R6.1, U2.6 (IO34)
- new net: R5.1, U2.8 (IO32)
- new net: SW3.1, U2.36 (IO22)
- new net: R4.1, SW3.2
- new net: D4.2 (A), R4.2
- new net: R2.1, SW1.2
- new net: D2.2 (A), R2.2
- new net: R3.1, SW2.2
- new net: D3.2 (A), R3.2
- new net: SW1.1, U2.23 (IO15)
- new net: SW2.1, U2.30 (IO18)
- new net: R7.2, U2.7 (IO35)
- new net +3.3V: U2.2 (VDD)
- new net ADC_I: R5.2
- new net ADC_R: R7.1
- new net ADC_V: R6.2
- new net GND: D2.1 (K), D3.1 (K), D4.1 (K), U2.1 (GND), U2.15 (GND), U2.38 (GND), U2.39 (GND)
Other:
- added sheet Resistance Measurement (resistance.kicad_sch)

Commit message: v1
Parts:
- removed R6, R7: 100R, symbol Device:R_Small
- removed SW3: SW_Push, symbol Switch:SW_Push
- removed U2: ESP32-WROOM-32, RF_Module:ESP32-WROOM-32, symbol RF_Module:ESP32-WROOM-32
- added C4, C5, C6: 0.1uF, symbol Device:C
- added J2: Conn_01x04_Pin, symbol Connector:Conn_01x04_Pin
- added NT1: NetTie_2, symbol Device:NetTie_2
- added R12, R13, R14: ~, symbol Device:R_Small
- added R15, R16: 2k, symbol Device:R_Small
- added SW3 (x2): SW_Push, symbol Switch:SW_Push
- added U3: PGA116AIPW, PW20, symbol PGA116:PGA116AIPW
- added U7: ESP32-S3-WROOM-1-N4, lab02_components:ESP32-S3-WROOM-1-N4, symbol lab02-symbols:ESP32-S3-WROOM-1-N4
- R2: footprint (none) -> Resistor_SMD:R_0603_1608Metric
Connections:
- net +3.3V: now also C4.1, C5.1, C6.1, J2.3 (Pin_3), R15.2, R16.2, U3.1 (AVDD), U3.19 (DVDD), U7.2 (3V3)
- net GND: now also C4.2, C5.2, C6.2, J2.4 (Pin_4), NT1.1, U3.14 (GND), U7.1 (GND)
- net at R5.1: now also U7.5 (IO5)
- net at R4.1: now also SW3.2, SW3.2
- net at R4.2: now also D2.2 (A); no longer D4.2 (A)
- net at R2.2: now also D4.2 (A); no longer D2.2 (A)
- net at SW1.1: now also U7.22 (IO14)
- net at SW2.1: now also U7.19 (IO11)
- net ADC_I renamed pga-v_o-adc
- net pga-v_o-adc: now also U3.9 (VOUT)
- new net: J2.1 (Pin_1), R16.1, U7.28 (IO35)
- new net: NT1.2, U3.8 (VREF)
- new net: J2.2 (Pin_2), R15.1, U7.29 (IO36)
- new net: SW3.1, SW3.1, U7.12 (IO8)
Other:
- added sheet Power Supply (power.kicad_sch)
- sheet Current Measurement ports: added PGA_I; removed none
- sheet Resistance Measurement ports: added PGA_R; removed none
- sheet Voltage Measurement ports: added PGA_V; removed none

Commit message: v2
Parts:
- removed D4: GREEN LED, LED_SMD:LED_0603_1608Metric_Pad1.05x0.95mm_HandSolder, symbol Device:LED
- removed SW3 (x2): SW_Push, symbol Switch:SW_Push
- added D5: GREEN LED, LED_SMD:LED_0603_1608Metric_Pad1.05x0.95mm_HandSolder, symbol Device:LED
- added SW4: SW_Push, symbol Switch:SW_Push
- R12, R14: value ~ -> 10k; now fitted
- R13: value ~ -> 2k; now fitted
- R2: value 56R -> 2k; footprint Resistor_SMD:R_0603_1608Metric -> (none)
- R3: value 56R -> 10k
- R4: value 56R -> 2k
Connections:
- net +3.3V: now also SW1.2, SW2.2, SW4.2
- net GND: now also R12.2, R14.2, R3.2, D5.1 (K)
- net pga_i: now also U3.2 (CH5)
- net pga_r: now also U3.6 (CH1)
- net pga_v: now also U3.4 (CH3)
- net at D2.2 (A): now also R2.2; no longer R4.2
- net SDA: now reaches J2.1 (Pin_1), R16.1
- net SDA: now also U7.21 (IO13); no longer U7.28 (IO35)
- net at R14.1: now also R4.1, SW2.1, U7.20 (IO12)
- net SCL: now reaches J2.2 (Pin_2), R15.1
- net SCL: now also U7.22 (IO14); no longer U7.29 (IO36)
- net at R12.1: now also R13.1, U7.12 (IO8), SW4.1
- net at D3.2 (A): now also R4.2; no longer R3.2
- net at SW1.1: now also R2.1, R3.1, U7.18 (IO10); no longer U7.22 (IO14)
- net at U7.19 (IO11): no longer SW2.1
- net at R13.2: now also D5.2 (A)
Other:
- sheet Current Measurement ports: added P-, P_I+; removed none
- sheet Resistance Measurement ports: added P-, P_R+; removed none
- sheet Voltage Measurement ports: added P-, P_V+; removed none
- moved on the sheet: C4, C5, C6, J2, NT1, R15, R16, R5, U3, U7

Commit message: v3
Parts:
- U7: Digikey PN (none) -> 1965-ESP32-S3-WROOM-1-N4CT-ND; MPN (none) -> ESP32-S3-WROOM-1-N4
Changed lines of the file:
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@@
       (effects (font (size 1.27 1.27)) (justify bottom) hide)
+    )
+    (property "Digikey PN" "1965-ESP32-S3-WROOM-1-N4CT-ND" (at 181.61 68.58 0)
+      (effects (font (size 1.27 1.27)) hide)
+    )
+    (property "MPN" "ESP32-S3-WROOM-1-N4" (at 181.61 68.58 0)
+      (effects (font (size 1.27 1.27)) hide)
     )
     (pin "5")

Commit message: v4
Parts:
- added C8: 1uF, Capacitor_SMD:C_0603_1608Metric, symbol Device:C
- added J3: USB_C_Receptacle_USB2.0_14P, symbol Connector:USB_C_Receptacle_USB2.0_14P
- added R17: 442K, Resistor_SMD:R_0603_1608Metric, symbol Device:R_Small
- added R18: 160K, Resistor_SMD:R_0603_1608Metric, symbol Device:R_Small
- added R19, R20, R21: 5.1K, Resistor_SMD:R_0603_1608Metric, symbol Device:R_Small
- added SW3, SW5: SW_MEC_5E, symbol Switch:SW_MEC_5E
- C4, C5, C6: footprint (none) -> Capacitor_SMD:C_0603_1608Metric
- R12, R14, R3: value 10k -> 10K; footprint (none) -> Resistor_SMD:R_0603_1608Metric
- R13, R15, R16, R2, R4: value 2k -> 2K; footprint (none) -> Resistor_SMD:R_0603_1608Metric
- R5: footprint (none) -> Resistor_SMD:R_0603_1608Metric
Connections:
- net +3.3V: now also R19.1
- net GND: now also C8.2, J3.A1 (GND), J3.A12 (GND), J3.B1 (GND), J3.B12 (GND), J3.S1 (SHIELD), R18.1, R20.2, R21.2, SW3.1, SW3.2, SW5.1, SW5.2
- net USB_N: now reaches U7.13 (IO19)
- net USB_N: now also J3.A7 (D-), J3.B7 (D-)
- net USB_P: now reaches U7.14 (IO20)
- net USB_P: now also J3.A6 (D+), J3.B6 (D+)
- net boot: now reaches U7.27 (IO0)
- net boot: now also SW3.3 (K), SW3.4 (A)
- net reset: now reaches U7.3 (EN)
- net reset: now also SW5.4 (A)
- net at U7.39 (IO1): now also R17.1, R18.2
- new net: C8.1, R19.2, SW5.3 (K)
- new net: J3.A5 (CC1), R20.1
- new net: J3.B5 (CC2), R21.1
- new net: J3.A4 (VBUS), J3.A9 (VBUS), J3.B4 (VBUS), J3.B9 (VBUS)
- new net vbat: R17.2
- no-connect marks 0 -> 1
Other:
- sheet Power Supply ports: added VBAT; removed none
- moved on the sheet: J2, R15, R16

Commit message: v5
Parts:
- J3: footprint (none) -> lab02_components:USB4085-GF-A; Digikey PN (none) -> 2073-USB4085-GF-ACT-ND; MPN (none) -> USB4085-GF-A
Changed lines of the file:
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@@
       (effects (font (size 1.27 1.27)))
     )
-    (property "Footprint" "" (at 236.22 129.54 0)
+    (property "Footprint" "lab02_components:USB4085-GF-A" (at 236.22 129.54 0)
       (effects (font (size 1.27 1.27)) hide)
     )
-    (property "Datasheet" "https://www.usb.org/sites/default/files/documents/usb_type-c.zip" (at 236.22 129.54 0)
+    (property "Datasheet" "https://gct.co/files/drawings/usb4085.pdf" (at 236.22 129.54 0)
       (effects (font (size 1.27 1.27)) hide)
     )
+    (property "Digikey PN" "2073-USB4085-GF-ACT-ND" (at 232.41 129.54 0)
+      (effects (font (size 1.27 1.27)) hide)
+    )
+    (property "MPN" "USB4085-GF-A" (at 232.41 129.54 0)
+      (effects (font (size 1.27 1.27)) hide)
+    )

Commit message: v6
Parts:
- SW1, SW2, SW4: footprint (none) -> lab02_components:SWITCH_FSMSM_TYC; Digikey PN (none) -> 450-1140-ND; MPN (none) -> FSMSM
- U3: footprint PW20 -> lab02_components:PGA116AIPWR; Digikey PN (none) -> 296-23772-1-ND; MPN (none) -> PGA116AIPWR
Changed lines of the file:
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@@
       (effects (font (size 1.524 1.524)))
     )
-    (property "Footprint" "PW20" (at 50.8 168.91 0)
+    (property "Footprint" "lab02_components:PGA116AIPWR" (at 50.8 168.91 0)
       (effects (font (size 1.27 1.27) italic) hide)
     )
-    (property "Datasheet" "PGA116AIPW" (at 50.8 168.91 0)
+    (property "Datasheet" "https://www.ti.com/lit/ds/symlink/pga112.pdf?HQS=dis-dk-null-digikeymode-dsf-pf-null-wwe&ts=1705418851270&ref_url=https%253A%252F%252Fwww.ti.com%252Fgeneral%252Fdocs%252Fsuppproductinfo.tsp%253FdistId%253D10%2526gotoUrl%253Dhttps%253A%252F%252Fwww.ti.com%252Flit%252Fgpn%252Fpga112" (at 50.8 168.91 0)
       (effects (font (size 1.27 1.27) italic) hide)
+    )
+    (property "Digikey PN" "296-23772-1-ND" (at 50.8 168.91 0)
+      (effects (font (size 1.27 1.27)) hide)
+    )
+    (property "MPN" "PGA116AIPWR" (at 50.8 168.91 0)
+      (effects (font (size 1.27 1.27)) hide)
     )
     (pin "10")
@@
       (effects (font (size 1.27 1.27)) (justify right))
     )
-    (property "Footprint" "" (at 109.22 45.72 0)
+    (property "Footprint" "lab02_components:SWITCH_FSMSM_TYC" (at 109.22 45.72 0)
       (effects (font (size 1.27 1.27)) hide)
     )
@@
       (effects (font (size 1.27 1.27)) hide)
     )
-    (property "Digikey PN" "" (at 114.3 45.72 0)
-      (effects (font (size 1.27 1.27)) hide)
-    )
-    (property "MPN" "" (at 114.3 45.72 0)
+    (property "Digikey PN" "450-1140-ND" (at 114.3 45.72 0)
+      (effects (font (size 1.27 1.27)) hide)
+    )
+    (property "MPN" "FSMSM" (at 114.3 45.72 0)
       (effects (font (size 1.27 1.27)) hide)
     )
@@
       (effects (font (size 1.27 1.27)) (justify right))
     )
-    (property "Footprint" "" (at 133.35 97.79 0)
+    (property "Footprint" "lab02_components:SWITCH_FSMSM_TYC" (at 133.35 97.79 0)
       (effects (font (size 1.27 1.27)) hide)
     )
@@
       (effects (font (size 1.27 1.27)) hide)
     )
-    (property "Digikey PN" "" (at 138.43 97.79 0)
-      (effects (font (size 1.27 1.27)) hide)
-    )
-    (property "MPN" "" (at 138.43 97.79 0)
+    (property "Digikey PN" "450-1140-ND" (at 138.43 97.79 0)
+      (effects (font (size 1.27 1.27)) hide)
+    )
+    (property "MPN" "FSMSM" (at 138.43 97.79 0)
       (effects (font (size 1.27 1.27)) hide)
     )
@@
       (effects (font (size 1.27 1.27)) (justify right))
     )
-    (property "Footprint" "" (at 109.22 83.82 0)
+    (property "Footprint" "lab02_components:SWITCH_FSMSM_TYC" (at 109.22 83.82 0)
       (effects (font (size 1.27 1.27)) hide)
     )
@@
       (effects (font (size 1.27 1.27)) hide)
     )
-    (property "Digikey PN" "" (at 114.3 83.82 0)
-      (effects (font (size 1.27 1.27)) hide)
-    )
-    (property "MPN" "" (at 114.3 83.82 0)
-      (effects (font (size 1.27 1.27)) hide)
-    )
+    (property "Digikey PN" "450-1140-ND" (at 114.3 83.82 0)
+      (effects (font (size 1.27 1.27)) hide)
+    )
+    (property "MPN" "FSMSM" (at 114.3 83.82 0)
+      (effects (font (size 1.27 1.27)) hide)
+    )

Commit message: v7
Parts:
- removed C8: 1uF, Capacitor_SMD:C_0603_1608Metric, symbol Device:C
- removed R19: 5.1K, Resistor_SMD:R_0603_1608Metric, symbol Device:R_Small
- removed SW3, SW5: SW_MEC_5E, symbol Switch:SW_MEC_5E
- added C9: 1uF, Capacitor_SMD:C_0603_1608Metric, symbol Device:C
- added R22: 10K, Resistor_SMD:R_0603_1608Metric, symbol Device:R_Small
- added R23: 5.1K, Resistor_SMD:R_0603_1608Metric, symbol Device:R_Small
- added SW3, SW5: SW_SPST, lab02_components:SWITCH_FSMSM_TYC, symbol Switch:SW_Push
- J2: footprint (none) -> lab02_components:PPTC041LFBN-RC; Digikey PN (none) -> S7002-ND; MPN (none) -> PPTC041LFBN-RC
- SW1, SW2, SW4: value SW_Push -> SW_SPST
Connections:
- net +3.3V: now also R23.1
- net GND: now also U7.40 (GND__1), U7.41_1 (GND__2), U7.41_2 (GND__3), U7.41_3 (GND__4), U7.41_4 (GND__5), U7.41_5 (GND__6), U7.41_6 (GND__7), U7.41_7 (GND__8), U7.41_8 (GND__9), U7.41_9 (GND__10), C9.2, SW3.1, SW5.1
- net boot: now also R22.2
- net reset: now also C9.1, R23.2, SW3.2
- net SCLK: now reaches U3.15 (SCLK)
- net SCLK: now also U7.31 (IO38)
- net SDO_ESP-SDI_PGA: now reaches U3.16 (DIN)
- net SDO_ESP-SDI_PGA: now also U7.29 (IO36)
- net SDI_ESP-SDO_PGA: now reaches U3.17 (DOUT)
- net SDI_ESP-SDO_PGA: now also U7.30 (IO37)
- net ~{CS}: now reaches U3.18 (*CS)
- net ~{CS}: now also U7.28 (IO35)
- new net: R22.1, SW5.2
Other:
- moved on the sheet: C5
