File: lab02/lab02.kicad_sch (KiCad schematic)
At the start: 32 parts, among them J2 Conn_01x04_Pin, J3 USB_C_Receptacle_USB2.0_14P, SW1 SW_SPST, SW2 SW_SPST, SW3 SW_SPST, SW4 SW_SPST, SW5 SW_SPST, U3 PGA116AIPW, U7 ESP32-S3-WROOM-1-N4

Commit message: pcb layout v0
Parts:
- added J4, J5: FCR7350R, CONN1_FCR7350R_CLF, symbol lab02-symbols:FCR7350(banana-jack)
- added J6: FCR7350B, CONN1_FCR7350R_CLF, symbol lab02-symbols:FCR7350(banana-jack)
- NT1: footprint (none) -> NetTie:NetTie-2_SMD_Pad0.5mm
- renumbered SW4 to SW3, SW3 to SW4
Connections:
- net vusb: now reaches J3.A4 (VBUS), J3.A9 (VBUS), J3.B4 (VBUS), J3.B9 (VBUS)
- new net p+_i: J5.1
- new net p+_v-r: J4.1
- new net p-: J6.1
- no-connect marks 1 -> 0
Other:
- sheet Power Supply ports: added VUSB; removed none

Commit message: v3
Connections:
- net at R14.1, R4.1, SW2.1: now also U7.18 (IO10); no longer U7.20 (IO12)
- net at R2.1, R3.1, SW1.1: now also U7.20 (IO12); no longer U7.18 (IO10)
- net at R12.1, R13.1, SW3.1: now also U7.17 (IO9); no longer U7.12 (IO8)
Changed lines of the file:
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@@
-    (stroke (width 0) (type default))
-  )
-  (wire (pts (xy 127 73.66) (xy 166.37 73.66))
     (stroke (width 0) (type default))
   )
@@
     (stroke (width 0) (type default))
   )
-  (wire (pts (xy 158.75 102.87) (xy 138.43 102.87))
+  (wire (pts (xy 152.4 102.87) (xy 138.43 102.87))
     (stroke (width 0) (type default))
   )
@@
     (stroke (width 0) (type default))
   )
+  (wire (pts (xy 152.4 78.74) (xy 166.37 78.74))
+    (stroke (width 0) (type default))
+  )
   (wire (pts (xy 55.88 38.1) (xy 62.23 38.1))
     (stroke (width 0) (type default))
@@
     (stroke (width 0) (type default))
   )
-  (wire (pts (xy 158.75 83.82) (xy 158.75 102.87))
+  (wire (pts (xy 152.4 78.74) (xy 152.4 102.87))
     (stroke (width 0) (type default))
   )
@@
   )
   (wire (pts (xy 243.84 44.45) (xy 245.11 44.45))
+    (stroke (width 0) (type default))
+  )
+  (wire (pts (xy 127 76.2) (xy 166.37 76.2))
     (stroke (width 0) (type default))
   )
@@
     (stroke (width 0) (type default))
   )
-  (wire (pts (xy 158.75 83.82) (xy 166.37 83.82))
-    (stroke (width 0) (type default))
-  )
   (wire (pts (xy 151.13 171.45) (xy 158.75 171.45))
     (stroke (width 0) (type default))
@@
     (stroke (width 0) (type default))
   )
-  (wire (pts (xy 247.65 127) (xy 247.65 129.54))
+  (wire (pts (xy 127 50.8) (xy 127 76.2))
     (stroke (width 0) (type default))
   )
-  (wire (pts (xy 127 78.74) (xy 166.37 78.74))
+  (wire (pts (xy 247.65 127) (xy 247.65 129.54))
     (stroke (width 0) (type default))
   )
@@
     (stroke (width 0) (type default))
   )
-  (wire (pts (xy 127 88.9) (xy 127 78.74))
+  (wire (pts (xy 127 88.9) (xy 127 83.82))
     (stroke (width 0) (type default))
   )
@@
     (stroke (width 0) (type default))
   )
-  (wire (pts (xy 127 50.8) (xy 127 73.66))
-    (stroke (width 0) (type default))
-  )
   (wire (pts (xy 196.85 119.38) (xy 196.85 116.84))
     (stroke (width 0) (type default))
@@
     (stroke (width 0) (type default))
   )
+  (wire (pts (xy 127 83.82) (xy 166.37 83.82))
+    (stroke (width 0) (type default))
+  )

Commit message: v7 pcb
Parts:
- removed R17: 442K, Resistor_SMD:R_0603_1608Metric, symbol Device:R_Small
- removed R18: 160K, Resistor_SMD:R_0603_1608Metric, symbol Device:R_Small
Connections:
- net SCL: now also U7.24 (IO47); no longer U7.22 (IO14)
- net SDA: now also U7.25 (IO48); no longer U7.21 (IO13)
- net SDI_ESP-SDO_PGA: now also U7.29 (IO36); no longer U7.30 (IO37)
- net SDO_ESP-SDI_PGA: now also U7.30 (IO37); no longer U7.29 (IO36)
- net pga-v_o-adc: now also R5.1; no longer R5.2
- net at R14.1, SW2.1, U7.18 (IO10): no longer R4.1
- net at R3.1, SW1.1, U7.20 (IO12): no longer R2.1
- net at R12.1, SW3.1: now also U7.15 (IO3); no longer R13.1, U7.17 (IO9)
- net at U7.19 (IO11): now also R4.1
- net at U7.38 (IO2): now also R5.2
- net at U7.5 (IO5): no longer R5.1
- new net: R2.1, U7.21 (IO13)
- new net: R13.1, U7.17 (IO9)
Other:
- moved on the sheet: D2, D3, D5, J4, J5, J6, R12, R13, R14, R2, R3, R4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

Commit message: v8
Parts:
- added H1, H2, H3, H4: MountingHole, MountingHole:MountingHole_2.5mm, symbol Mechanical:MountingHole
- J3: footprint lab02_components:USB4085-GF-A -> Connector_USB:USB_C_Receptacle_GCT_USB4085
- U7: footprint lab02_components:ESP32-S3-WROOM-1-N4 -> RF_Module:ESP32-S3-WROOM-1
Connections:
- net GND: now also U7.41 (GND__2); no longer U7.41_1 (GND__2)
Changed lines of the file:
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@@
+    )
+  )
+  (symbol (lib_id "Mechanical:MountingHole") (at 74.93 26.67 0) (unit 1)
+    (in_bom yes) (on_board yes) (dnp no) (fields_autoplaced)
+    (property "Reference" "H2" (at 77.47 25.4 0)
+      (effects (font (size 1.27 1.27)) (justify left))
+    )
+    (property "Value" "MountingHole" (at 77.47 27.94 0)
+      (effects (font (size 1.27 1.27)) (justify left))
+    )
+    (property "Footprint" "MountingHole:MountingHole_2.5mm" (at 74.93 26.67 0)
+      (effects (font (size 1.27 1.27)) hide)
+    )
+    (property "Datasheet" "~" (at 74.93 26.67 0)
+      (effects (font (size 1.27 1.27)) hide)
+    )
+    (instances
+      (project "lab02"
+        (path "/352d7abe-fc72-4473-8b68-62eecf44f496"
+          (reference "H2") (unit 1)
+        )
+      )
     )
   )
@@
       (effects (font (size 1.27 1.27)))
     )
-    (property "Footprint" "lab02_components:USB4085-GF-A" (at 236.22 129.54 0)
+    (property "Footprint" "Connector_USB:USB_C_Receptacle_GCT_USB4085" (at 236.22 129.54 0)
       (effects (font (size 1.27 1.27)) hide)
     )
@@
     )
   )
+  (symbol (lib_id "Mechanical:MountingHole") (at 96.52 19.05 0) (unit 1)
+    (in_bom yes) (on_board yes) (dnp no) (fields_autoplaced)
+    (property "Reference" "H3" (at 99.06 17.78 0)
+      (effects (font (size 1.27 1.27)) (justify left))
+    )
+    (property "Value" "MountingHole" (at 99.06 20.32 0)
+      (effects (font (size 1.27 1.27)) (justify left))
+    )
+    (property "Footprint" "MountingHole:MountingHole_2.5mm" (at 96.52 19.05 0)
+      (effects (font (size 1.27 1.27)) hide)
+    )
+    (property "Datasheet" "~" (at 96.52 19.05 0)
+      (effects (font (size 1.27 1.27)) hide)
+    )
+    (instances
+      (project "lab02"
+        (path "/352d7abe-fc72-4473-8b68-62eecf44f496"
+          (reference "H3") (unit 1)
+        )
+      )
+    )
+  )
   (symbol (lib_id "power:GND") (at 99.06 92.71 0) (unit 1)
     (in_bom yes) (on_board yes) (dnp no) (fields_autoplaced)
@@
         (path "/352d7abe-fc72-4473-8b68-62eecf44f496"
           (reference "SW5") (unit 1)
+        )
+      )
+    )
+  )
+  (symbol (lib_id "Mechanical:MountingHole") (at 74.93 19.05 0) (unit 1)
+    (in_bom yes) (on_board yes) (dnp no) (fields_autoplaced)
+    (property "Reference" "H1" (at 77.47 17.78 0)
+      (effects (font (size 1.27 1.27)) (justify left))
+    )
+    (property "Value" "MountingHole" (at 77.47 20.32 0)
+      (effects (font (size 1.27 1.27)) (justify left))
+    )
+    (property "Footprint" "MountingHole:MountingHole_2.5mm" (at 74.93 19.05 0)
+      (effects (font (size 1.27 1.27)) hide)
+    )
+    (property "Datasheet" "~" (at 74.93 19.05 0)
+      (effects (font (size 1.27 1.27)) hide)
+    )
+    (instances
+      (project "lab02"
+        (path "/352d7abe-fc72-4473-8b68-62eecf44f496"
+          (reference "H1") (unit 1)
         )
       )
@@
       (effects (font (size 1.27 1.27)))
     )
-    (property "Footprint" "lab02_components:ESP32-S3-WROOM-1-N4" (at 181.61 68.58 0)
+    (property "Footprint" "RF_Module:ESP32-S3-WROOM-1" (at 181.61 68.58 0)
       (effects (font (size 1.27 1.27)) (justify bottom) hide)
     )
@@
     (pin "13")
     (pin "7")
-    (pin "41_1")
+    (pin "41")
     (pin "8")
     (pin "41_2")
@@
         )
       )
+    )
+  )
+  (symbol (lib_id "Mechanical:MountingHole") (at 96.52 26.67 0) (unit 1)
+    (in_bom yes) (on_board yes) (dnp no) (fields_autoplaced)
+    (property "Reference" "H4" (at 99.06 25.4 0)
+      (effects (font (size 1.27 1.27)) (justify left))
+    )
+    (property "Value" "MountingHole" (at 99.06 27.94 0)
+      (effects (font (size 1.27 1.27)) (justify left))
+    )
+    (property "Footprint" "MountingHole:MountingHole_2.5mm" (at 96.52 26.67 0)
+      (effects (font (size 1.27 1.27)) hide)
+    )
+    (property "Datasheet" "~" (at 96.52 26.67 0)
+      (effects (font (size 1.27 1.27)) hide)
+    )
+    (instances
+      (project "lab02"
+        (path "/352d7abe-fc72-4473-8b68-62eecf44f496"
+          (reference "H4") (unit 1)
+        )
+      )

Commit message: v9
Parts:
- added H5: logo1, lab02_components:EdgertonLogo, symbol Mechanical:MountingHole
- added H6: logo2, lab02_components:EECSLogo, symbol Mechanical:MountingHole
- added H7: logo1, lab02_components:MechE, symbol Mechanical:MountingHole
Changed lines of the file:
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@@
+    )
+  )
+  (symbol (lib_id "Mechanical:MountingHole") (at 152.4 22.86 0) (unit 1)
+    (in_bom yes) (on_board yes) (dnp no) (fields_autoplaced)
+    (property "Reference" "H6" (at 154.94 21.59 0)
+      (effects (font (size 1.27 1.27)) (justify left))
+    )
+    (property "Value" "logo2" (at 154.94 24.13 0)
+      (effects (font (size 1.27 1.27)) (justify left))
+    )
+    (property "Footprint" "lab02_components:EECSLogo" (at 152.4 22.86 0)
+      (effects (font (size 1.27 1.27)) hide)
+    )
+    (property "Datasheet" "~" (at 152.4 22.86 0)
+      (effects (font (size 1.27 1.27)) hide)
+    )
+    (instances
+      (project "lab02"
+        (path "/352d7abe-fc72-4473-8b68-62eecf44f496"
+          (reference "H6") (unit 1)
+        )
+      )
     )
   )
@@
     )
   )
+  (symbol (lib_id "Mechanical:MountingHole") (at 130.81 22.86 0) (unit 1)
+    (in_bom yes) (on_board yes) (dnp no) (fields_autoplaced)
+    (property "Reference" "H5" (at 133.35 21.59 0)
+      (effects (font (size 1.27 1.27)) (justify left))
+    )
+    (property "Value" "logo1" (at 133.35 24.13 0)
+      (effects (font (size 1.27 1.27)) (justify left))
+    )
+    (property "Footprint" "lab02_components:EdgertonLogo" (at 130.81 22.86 0)
+      (effects (font (size 1.27 1.27)) hide)
+    )
+    (property "Datasheet" "~" (at 130.81 22.86 0)
+      (effects (font (size 1.27 1.27)) hide)
+    )
+    (instances
+      (project "lab02"
+        (path "/352d7abe-fc72-4473-8b68-62eecf44f496"
+          (reference "H5") (unit 1)
+        )
+      )
+    )
+  )
   (symbol (lib_id "Mechanical:MountingHole") (at 96.52 19.05 0) (unit 1)
     (in_bom yes) (on_board yes) (dnp no) (fields_autoplaced)
@@
         )
       )
+    )
+  )
+  (symbol (lib_id "Mechanical:MountingHole") (at 143.51 30.48 0) (unit 1)
+    (in_bom yes) (on_board yes) (dnp no) (fields_autoplaced)
+    (property "Reference" "H7" (at 146.05 29.21 0)
+      (effects (font (size 1.27 1.27)) (justify left))
+    )
+    (property "Value" "logo1" (at 146.05 31.75 0)
+      (effects (font (size 1.27 1.27)) (justify left))
+    )
+    (property "Footprint" "lab02_components:MechE" (at 143.51 30.48 0)
+      (effects (font (size 1.27 1.27)) hide)
+    )
+    (property "Datasheet" "~" (at 143.51 30.48 0)
+      (effects (font (size 1.27 1.27)) hide)
+    )
+    (instances
+      (project "lab02"
+        (path "/352d7abe-fc72-4473-8b68-62eecf44f496"
+          (reference "H7") (unit 1)
+        )
+      )
