File: lab02/resistance.kicad_sch (KiCad schematic)
At the start: 2 parts

Commit message: v1
Parts:
- added U1: OPA310 DBV, lab02_components:SOT-23-5-DBV_TEX, symbol Amplifier_Operational:OPA188xxDBV
- D1: value D_Zener -> 3.3V; Digikey PN (none) -> 3757-BZT52-C3V3_R1_00001CT-ND
- R1: footprint (none) -> Resistor_SMD:R_0603_1608Metric
Connections:
- net +3.3V: now also R1.1, U1.5 (V+)
- net GND: now also D1.2 (A), U1.2 (V-); no longer D1.1 (K), R1.2
- removed net P-: D1.2 (A), R1.1
- new net PGA_R: U1.1, U1.4 (-)
- new net P_R+: D1.1 (K), R1.2, U1.3 (+)
Other:
- moved on the sheet: D1

Commit message: v2
Changed lines of the file:
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@@
     (stroke (width 0) (type default))
-  )
-  (global_label "P-" (shape input) (at 146.05 95.25 0) (fields_autoplaced)
-    (effects (font (size 1.27 1.27)) (justify left))
-    (property "Intersheetrefs" "${INTERSHEET_REFS}" (at 151.8776 95.25 0)
-      (effects (font (size 1.27 1.27)) (justify left) hide)
-    )
-  )
-  (global_label "P_R+" (shape input) (at 146.05 87.63 0) (fields_autoplaced)
-    (effects (font (size 1.27 1.27)) (justify left))
-    (property "Intersheetrefs" "${INTERSHEET_REFS}" (at 154.1152 87.63 0)
-      (effects (font (size 1.27 1.27)) (justify left) hide)
-    )
   )
   (hierarchical_label "PGA_R" (shape input) (at 104.14 85.09 180) (fields_autoplaced)
     (effects (font (size 1.27 1.27)) (justify right))
   )
+  (hierarchical_label "P_R+" (shape input) (at 146.05 87.63 0) (fields_autoplaced)
+    (effects (font (size 1.27 1.27)) (justify left))
+  )
+  (hierarchical_label "P-" (shape input) (at 146.05 95.25 0) (fields_autoplaced)
+    (effects (font (size 1.27 1.27)) (justify left))
+  )
   (symbol (lib_id "power:+3.3V") (at 114.3 92.71 0) (unit 1)

Commit message: v3
Parts:
- U1: value OPA310 DBV -> OPA310IDBVR; footprint lab02_components:SOT-23-5-DBV_TEX -> lab02_components:OPA310IDBVR; Digikey PN (none) -> 296-OPA310IDBVRCT-ND; MPN (none) -> OPA310IDBVR
Changed lines of the file:
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@@
       (effects (font (size 1.27 1.27)) (justify right))
     )
-    (property "Value" "OPA310 DBV" (at 119.7259 77.47 0)
+    (property "Value" "OPA310IDBVR" (at 119.7259 77.47 0)
       (effects (font (size 1.27 1.27)) (justify right))
     )
-    (property "Footprint" "lab02_components:SOT-23-5-DBV_TEX" (at 116.84 85.09 0)
+    (property "Footprint" "lab02_components:OPA310IDBVR" (at 116.84 85.09 0)
       (effects (font (size 1.27 1.27)) hide)
     )
-    (property "Datasheet" "https://www.ti.com/lit/ds/symlink/opa310.pdf?ts=1705006057026&ref_url=https%253A%252F%252Fwww.ti.com%252Fproduct%252FOPA310" (at 116.84 90.17 0)
+    (property "Datasheet" "https://www.ti.com/lit/ds/symlink/opa310.pdf" (at 116.84 90.17 0)
       (effects (font (size 1.27 1.27)) hide)
     )
+    (property "Digikey PN" "296-OPA310IDBVRCT-ND" (at 116.84 85.09 0)
+      (effects (font (size 1.27 1.27)) hide)
+    )
+    (property "MPN" "OPA310IDBVR" (at 116.84 85.09 0)
+      (effects (font (size 1.27 1.27)) hide)
+    )

Commit message: v4
Parts:
- R1: value 100k -> 100K
Changed lines of the file:
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@@
       (effects (font (size 1.27 1.27)) (justify left))
     )
-    (property "Value" "100k" (at 142.24 81.28 0)
+    (property "Value" "100K" (at 142.24 81.28 0)
       (effects (font (size 1.27 1.27)) (justify left))
     )

Commit message: v7
Parts:
- added C10: 100nF, Capacitor_SMD:C_0603_1608Metric, symbol Device:C
- D1: footprint (none) -> lab02_components:MMSZ4684T1G; Digikey PN 3757-BZT52-C3V3_R1_00001CT-ND -> MMSZ4684T1GOSCT-ND; MPN (none) -> MMSZ4684T1G
Connections:
- net +3.3V: now also C10.1
- net GND: now also C10.2
Changed lines of the file:
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@@
   (junction (at 128.27 87.63) (diameter 0) (color 0 0 0 0)
   )
+  (junction (at 116.84 92.71) (diameter 0) (color 0 0 0 0)
+  )
   (junction (at 128.27 95.25) (diameter 0) (color 0 0 0 0)
   )
@@
     (stroke (width 0) (type default))
   )
-  (wire (pts (xy 105.41 95.25) (xy 128.27 95.25))
-    (stroke (width 0) (type default))
-  )
   (wire (pts (xy 114.3 73.66) (xy 119.38 73.66))
     (stroke (width 0) (type default))
   )
+  (wire (pts (xy 116.84 92.71) (xy 119.38 92.71))
+    (stroke (width 0) (type default))
+  )
   (wire (pts (xy 104.14 85.09) (xy 107.95 85.09))
     (stroke (width 0) (type default))
@@
     (stroke (width 0) (type default))
   )
+  (wire (pts (xy 124.46 95.25) (xy 128.27 95.25))
+    (stroke (width 0) (type default))
+  )
   (wire (pts (xy 107.95 78.74) (xy 107.95 85.09))
     (stroke (width 0) (type default))
   )
-  (wire (pts (xy 114.3 92.71) (xy 119.38 92.71))
+  (wire (pts (xy 114.3 92.71) (xy 116.84 92.71))
     (stroke (width 0) (type default))
   )
@@
   )
   (wire (pts (xy 124.46 78.74) (xy 107.95 78.74))
+    (stroke (width 0) (type default))
+  )
+  (wire (pts (xy 124.46 96.52) (xy 124.46 95.25))
     (stroke (width 0) (type default))
   )
@@
     )
   )
-  (symbol (lib_id "power:GND") (at 105.41 95.25 0) (unit 1)
-    (in_bom yes) (on_board yes) (dnp no) (fields_autoplaced)
-    (property "Reference" "#PWR02" (at 105.41 101.6 0)
-      (effects (font (size 1.27 1.27)) hide)
-    )
-    (property "Value" "GND" (at 105.41 100.33 0)
-      (effects (font (size 1.27 1.27)))
-    )
-    (property "Footprint" "" (at 105.41 95.25 0)
-      (effects (font (size 1.27 1.27)) hide)
-    )
-    (property "Datasheet" "" (at 105.41 95.25 0)
+  (symbol (lib_id "power:GND") (at 124.46 96.52 0) (unit 1)
+    (in_bom yes) (on_board yes) (dnp no) (fields_autoplaced)
+    (property "Reference" "#PWR02" (at 124.46 102.87 0)
+      (effects (font (size 1.27 1.27)) hide)
+    )
+    (property "Value" "GND" (at 124.46 101.6 0)
+      (effects (font (size 1.27 1.27)))
+    )
+    (property "Footprint" "" (at 124.46 96.52 0)
+      (effects (font (size 1.27 1.27)) hide)
+    )
+    (property "Datasheet" "" (at 124.46 96.52 0)
       (effects (font (size 1.27 1.27)) hide)
     )
@@
     )
   )
+  (symbol (lib_id "power:GND") (at 116.84 100.33 0) (unit 1)
+    (in_bom yes) (on_board yes) (dnp no) (fields_autoplaced)
+    (property "Reference" "#PWR044" (at 116.84 106.68 0)
+      (effects (font (size 1.27 1.27)) hide)
+    )
+    (property "Value" "GND" (at 116.84 105.41 0)
+      (effects (font (size 1.27 1.27)))
+    )
+    (property "Footprint" "" (at 116.84 100.33 0)
+      (effects (font (size 1.27 1.27)) hide)
+    )
+    (property "Datasheet" "" (at 116.84 100.33 0)
+      (effects (font (size 1.27 1.27)) hide)
+    )
+    (pin "1")
+    (instances
+      (project "lab02"
+        (path "/352d7abe-fc72-4473-8b68-62eecf44f496/80a2bdd5-68af-43db-8a34-2b7856ec04c6"
+          (reference "#PWR044") (unit 1)
+        )
+      )
+    )
+  )
   (symbol (lib_id "Device:D_Zener") (at 128.27 91.44 270) (unit 1)
     (in_bom yes) (on_board yes) (dnp no) (fields_autoplaced)
@@
       (effects (font (size 1.27 1.27)) (justify left))
     )
-    (property "Footprint" "" (at 128.27 91.44 0)
-      (effects (font (size 1.27 1.27)) hide)
-    )
-    (property "Datasheet" "~" (at 128.27 91.44 0)
-      (effects (font (size 1.27 1.27)) hide)
-    )
-    (property "Digikey PN" "3757-BZT52-C3V3_R1_00001CT-ND" (at 128.27 91.44 0)
-      (effects (font (size 1.27 1.27)) hide)
-    )
-    (property "MPN" "" (at 128.27 91.44 0)
+    (property "Footprint" "lab02_components:MMSZ4684T1G" (at 128.27 91.44 0)
+      (effects (font (size 1.27 1.27)) hide)
+    )
+    (property "Datasheet" "https://www.onsemi.com/pdf/datasheet/mmsz4678t1-d.pdf" (at 128.27 91.44 0)
+      (effects (font (size 1.27 1.27)) hide)
+    )
+    (property "Digikey PN" "MMSZ4684T1GOSCT-ND" (at 128.27 91.44 0)
+      (effects (font (size 1.27 1.27)) hide)
+    )
+    (property "MPN" "MMSZ4684T1G" (at 128.27 91.44 0)
       (effects (font (size 1.27 1.27)) hide)
     )
@@
         )
       )
+    )
+  )
+  (symbol (lib_id "Device:C") (at 116.84 96.52 0) (unit 1)
+    (in_bom yes) (on_board yes) (dnp no)
+    (property "Reference" "C10" (at 110.49 95.25 0)
+      (effects (font (size 1.27 1.27)) (justify left))
+    )
+    (property "Value" "100nF" (at 107.95 97.79 0)
+      (effects (font (size 1.27 1.27)) (justify left))
+    )
+    (property "Footprint" "Capacitor_SMD:C_0603_1608Metric" (at 117.8052 100.33 0)
+      (effects (font (size 1.27 1.27)) hide)
+    )
+    (property "Datasheet" "~" (at 116.84 96.52 0)
+      (effects (font (size 1.27 1.27)) hide)
+    )
+    (pin "2")
+    (pin "1")
+    (instances
+      (project "lab02"
+        (path "/352d7abe-fc72-4473-8b68-62eecf44f496/80a2bdd5-68af-43db-8a34-2b7856ec04c6"
+          (reference "C10") (unit 1)
+        )
+      )
