File: lab02/current.kicad_sch (KiCad schematic)
At the start: 0 parts

Commit message: v1
Parts:
- added C7: 0.1uF, symbol Device:C
- added F1: 10A Fuse, symbol Device:Fuse
- added R6: 1mR, symbol Device:R_Small
- added R7: 340R, symbol Device:R_Small
- added R9: 0R, symbol Device:R_Small
- added U2: INA823, D0008A_SOIC_TEX, symbol lab02-symbols:INA823
Connections:
- new net: F1.2, R6.1, U2.3 (+IN)
- new net: R9.1, U2.5 (REF)
- new net: R7.1, U2.1 (RG)
- new net: R7.2, U2.8 (RG)
- new net +3.3V: C7.1, U2.7 (+VS)
- new net GND: C7.2, R6.2, R9.2, U2.2 (-IN), U2.4 (-VS)
- new net PGA_I: U2.6 (OUT)
- new net P_I+: F1.1

Commit message: v2
Changed lines of the file:
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@@
     (stroke (width 0) (type default))
   )
-  (global_label "P-" (shape input) (at 96.52 97.79 180) (fields_autoplaced)
+  (hierarchical_label "P_I+" (shape input) (at 96.52 80.01 180) (fields_autoplaced)
     (effects (font (size 1.27 1.27)) (justify right))
-    (property "Intersheetrefs" "${INTERSHEET_REFS}" (at 90.6924 97.79 0)
-      (effects (font (size 1.27 1.27)) (justify right) hide)
-    )
   )
-  (global_label "P_I+" (shape input) (at 96.52 80.01 180) (fields_autoplaced)
+  (hierarchical_label "P-" (shape input) (at 96.52 97.79 180) (fields_autoplaced)
     (effects (font (size 1.27 1.27)) (justify right))
-    (property "Intersheetrefs" "${INTERSHEET_REFS}" (at 89.12 80.01 0)
-      (effects (font (size 1.27 1.27)) (justify right) hide)
-    )
   )
   (hierarchical_label "PGA_I" (shape input) (at 175.26 91.44 0) (fields_autoplaced)

Commit message: v4
Parts:
- C7: footprint (none) -> Capacitor_SMD:C_0603_1608Metric
- R7, R9: footprint (none) -> Resistor_SMD:R_0603_1608Metric
Changed lines of the file:
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@@
       (effects (font (size 1.27 1.27)) (justify left))
     )
-    (property "Footprint" "" (at 167.64 96.52 0)
+    (property "Footprint" "Resistor_SMD:R_0603_1608Metric" (at 167.64 96.52 0)
       (effects (font (size 1.27 1.27)) hide)
     )
@@
       (effects (font (size 1.27 1.27)))
     )
-    (property "Footprint" "" (at 147.32 72.39 0)
+    (property "Footprint" "Resistor_SMD:R_0603_1608Metric" (at 147.32 72.39 0)
       (effects (font (size 1.27 1.27)) hide)
     )
@@
       (effects (font (size 1.27 1.27)) (justify left))
     )
-    (property "Footprint" "" (at 192.7352 96.52 0)
+    (property "Footprint" "Capacitor_SMD:C_0603_1608Metric" (at 192.7352 96.52 0)
       (effects (font (size 1.27 1.27)) hide)
     )

Commit message: v7
Parts:
- U2: footprint D0008A_SOIC_TEX -> (none)
Changed lines of the file:
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@@
       (effects (font (size 1.524 1.524)))
     )
-    (property "Footprint" "D0008A_SOIC_TEX" (at 127 86.36 0)
+    (property "Footprint" "" (at 127 86.36 0)
       (effects (font (size 1.27 1.27) italic) hide)
     )
-    (property "Datasheet" "XINA823DR" (at 127 86.36 0)
+    (property "Datasheet" "" (at 127 86.36 0)
       (effects (font (size 1.27 1.27) italic) hide)
     )

Commit message: pcb layout v0
Parts:
- added F2: 10A fuse cylinder, symbol Device:Fuse
- F1: footprint (none) -> lab02_components:FUSE_31.8221_SCH; Digikey PN (none) -> 486-1260-ND; MPN (none) -> 0031.8221
- R6: footprint (none) -> lab02_components:CSNL1206FT1L00; Digikey PN (none) -> CSNL1206FT1L00CT-ND; MPN (none) -> CSNL1206FT1L00
- U2: footprint (none) -> Package_SO:SOIC-8_3.9x4.9mm_P1.27mm; Digikey PN (none) -> 296-INA823DTCT-ND; MPN (none) -> INA823DT
Changed lines of the file:
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@@
       (effects (font (size 1.27 1.27)) (justify left))
     )
-    (property "Footprint" "" (at 111.76 88.9 0)
-      (effects (font (size 1.27 1.27)) hide)
-    )
-    (property "Datasheet" "~" (at 111.76 88.9 0)
+    (property "Footprint" "lab02_components:CSNL1206FT1L00" (at 111.76 88.9 0)
+      (effects (font (size 1.27 1.27)) hide)
+    )
+    (property "Datasheet" "https://www.seielect.com/catalog/sei-csnl.pdf" (at 111.76 88.9 0)
+      (effects (font (size 1.27 1.27)) hide)
+    )
+    (property "Digikey PN" "CSNL1206FT1L00CT-ND" (at 111.76 88.9 0)
+      (effects (font (size 1.27 1.27)) hide)
+    )
+    (property "MPN" "CSNL1206FT1L00" (at 111.76 88.9 0)
       (effects (font (size 1.27 1.27)) hide)
     )
@@
       (effects (font (size 1.27 1.27)))
     )
-    (property "Footprint" "" (at 104.14 81.788 90)
-      (effects (font (size 1.27 1.27)) hide)
-    )
-    (property "Datasheet" "~" (at 104.14 80.01 0)
+    (property "Footprint" "lab02_components:FUSE_31.8221_SCH" (at 104.14 81.788 90)
+      (effects (font (size 1.27 1.27)) hide)
+    )
+    (property "Datasheet" "https://www.schurter.com/en/datasheet/typ_OGN_Pre-Assembled.pdf" (at 104.14 80.01 0)
+      (effects (font (size 1.27 1.27)) hide)
+    )
+    (property "Digikey PN" "486-1260-ND" (at 104.14 80.01 0)
+      (effects (font (size 1.27 1.27)) hide)
+    )
+    (property "MPN" "0031.8221" (at 104.14 80.01 0)
       (effects (font (size 1.27 1.27)) hide)
     )
@@
       (effects (font (size 1.524 1.524)))
     )
-    (property "Footprint" "" (at 127 86.36 0)
+    (property "Footprint" "Package_SO:SOIC-8_3.9x4.9mm_P1.27mm" (at 127 86.36 0)
       (effects (font (size 1.27 1.27) italic) hide)
     )
-    (property "Datasheet" "" (at 127 86.36 0)
+    (property "Datasheet" "https://www.ti.com/lit/ds/symlink/ina823.pdf" (at 127 86.36 0)
       (effects (font (size 1.27 1.27) italic) hide)
+    )
+    (property "Digikey PN" "296-INA823DTCT-ND" (at 127 86.36 0)
+      (effects (font (size 1.27 1.27)) hide)
+    )
+    (property "MPN" "INA823DT" (at 127 86.36 0)
+      (effects (font (size 1.27 1.27)) hide)
     )
     (pin "1")
@@
         )
       )
+    )
+  )
+  (symbol (lib_id "Device:Fuse") (at 105.41 63.5 90) (unit 1)
+    (in_bom yes) (on_board no) (dnp no) (fields_autoplaced)
+    (property "Reference" "F2" (at 105.41 58.42 90)
+      (effects (font (size 1.27 1.27)))
+    )
+    (property "Value" "10A fuse cylinder" (at 105.41 60.96 90)
+      (effects (font (size 1.27 1.27)))
+    )
+    (property "Footprint" "" (at 105.41 65.278 90)
+      (effects (font (size 1.27 1.27)) hide)
+    )
+    (property "Datasheet" "https://www.schurter.com/en/datasheet/typ_D1.pdf" (at 105.41 63.5 0)
+      (effects (font (size 1.27 1.27)) hide)
+    )
+    (property "Digikey PN" "486-1865-ND" (at 105.41 63.5 0)
+      (effects (font (size 1.27 1.27)) hide)
+    )
+    (property "MPN" "7010.3530" (at 105.41 63.5 0)
+      (effects (font (size 1.27 1.27)) hide)
+    )
+    (pin "2")
+    (pin "1")
+    (instances
+      (project "lab02"
+        (path "/352d7abe-fc72-4473-8b68-62eecf44f496/4978ea04-f56b-4750-95a9-071f57b2b22a"
+          (reference "F2") (unit 1)
+        )
+      )
