File: lab02/power.kicad_sch (KiCad schematic)
At the start: 4 parts, among them J1 Conn_01x02_Pin, U5 AP2112K-3.3

Commit message: v4
Parts:
- C2, C3: footprint (none) -> Capacitor_SMD:C_0603_1608Metric
Connections:
- net +4V renamed VBAT
Other:
- moved on the sheet: J1
Changed lines of the file:
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@@
   (junction (at 130.81 100.33) (diameter 0) (color 0 0 0 0)
   )
+  (junction (at 121.92 100.33) (diameter 0) (color 0 0 0 0)
+  )
+  (wire (pts (xy 121.92 95.25) (xy 121.92 100.33))
+    (stroke (width 0) (type default))
+  )
   (wire (pts (xy 130.81 104.14) (xy 130.81 100.33))
     (stroke (width 0) (type default))
   )
-  (wire (pts (xy 119.38 100.33) (xy 130.81 100.33))
-    (stroke (width 0) (type default))
-  )
-  (wire (pts (xy 104.14 100.33) (xy 110.49 100.33))
+  (wire (pts (xy 113.03 100.33) (xy 121.92 100.33))
     (stroke (width 0) (type default))
   )
@@
     (stroke (width 0) (type default))
   )
-  (wire (pts (xy 104.14 102.87) (xy 110.49 102.87))
-    (stroke (width 0) (type default))
-  )
-  (symbol (lib_id "power:GND") (at 110.49 102.87 0) (unit 1)
-    (in_bom yes) (on_board yes) (dnp no) (fields_autoplaced)
-    (property "Reference" "#PWR016" (at 110.49 109.22 0)
-      (effects (font (size 1.27 1.27)) hide)
-    )
-    (property "Value" "GND" (at 110.49 107.95 0)
-      (effects (font (size 1.27 1.27)))
-    )
-    (property "Footprint" "" (at 110.49 102.87 0)
-      (effects (font (size 1.27 1.27)) hide)
-    )
-    (property "Datasheet" "" (at 110.49 102.87 0)
+  (wire (pts (xy 121.92 100.33) (xy 130.81 100.33))
+    (stroke (width 0) (type default))
+  )
+  (wire (pts (xy 113.03 102.87) (xy 119.38 102.87))
+    (stroke (width 0) (type default))
+  )
+  (hierarchical_label "VBAT" (shape input) (at 121.92 95.25 0) (fields_autoplaced)
+    (effects (font (size 1.27 1.27)) (justify left))
+  )
+  (symbol (lib_id "power:GND") (at 119.38 102.87 0) (unit 1)
+    (in_bom yes) (on_board yes) (dnp no) (fields_autoplaced)
+    (property "Reference" "#PWR016" (at 119.38 109.22 0)
+      (effects (font (size 1.27 1.27)) hide)
+    )
+    (property "Value" "GND" (at 119.38 107.95 0)
+      (effects (font (size 1.27 1.27)))
+    )
+    (property "Footprint" "" (at 119.38 102.87 0)
+      (effects (font (size 1.27 1.27)) hide)
+    )
+    (property "Datasheet" "" (at 119.38 102.87 0)
       (effects (font (size 1.27 1.27)) hide)
     )
@@
       (effects (font (size 1.27 1.27)) (justify left))
     )
-    (property "Footprint" "" (at 162.2552 107.95 0)
+    (property "Footprint" "Capacitor_SMD:C_0603_1608Metric" (at 162.2552 107.95 0)
       (effects (font (size 1.27 1.27)) hide)
     )
@@
     )
   )
-  (symbol (lib_id "Connector:Conn_01x02_Pin") (at 99.06 100.33 0) (unit 1)
-    (in_bom yes) (on_board yes) (dnp no) (fields_autoplaced)
-    (property "Reference" "J1" (at 99.695 95.25 0)
-      (effects (font (size 1.27 1.27)))
-    )
-    (property "Value" "Conn_01x02_Pin" (at 99.695 97.79 0)
-      (effects (font (size 1.27 1.27)))
-    )
-    (property "Footprint" "" (at 99.06 100.33 0)
-      (effects (font (size 1.27 1.27)) hide)
-    )
-    (property "Datasheet" "~" (at 99.06 100.33 0)
+  (symbol (lib_id "Connector:Conn_01x02_Pin") (at 107.95 100.33 0) (unit 1)
+    (in_bom yes) (on_board yes) (dnp no) (fields_autoplaced)
+    (property "Reference" "J1" (at 108.585 95.25 0)
+      (effects (font (size 1.27 1.27)))
+    )
+    (property "Value" "Conn_01x02_Pin" (at 108.585 97.79 0)
+      (effects (font (size 1.27 1.27)))
+    )
+    (property "Footprint" "" (at 107.95 100.33 0)
+      (effects (font (size 1.27 1.27)) hide)
+    )
+    (property "Datasheet" "~" (at 107.95 100.33 0)
       (effects (font (size 1.27 1.27)) hide)
     )
@@
         (path "/352d7abe-fc72-4473-8b68-62eecf44f496/4087662f-8023-43e4-a97d-75c33092c189"
           (reference "#PWR021") (unit 1)
-        )
-      )
-    )
-  )
-  (symbol (lib_id "power:+4V") (at 119.38 100.33 0) (unit 1)
-    (in_bom yes) (on_board yes) (dnp no) (fields_autoplaced)
-    (property "Reference" "#PWR019" (at 119.38 104.14 0)
-      (effects (font (size 1.27 1.27)) hide)
-    )
-    (property "Value" "+4V" (at 119.38 95.25 0)
-      (effects (font (size 1.27 1.27)))
-    )
-    (property "Footprint" "" (at 119.38 100.33 0)
-      (effects (font (size 1.27 1.27)) hide)
-    )
-    (property "Datasheet" "" (at 119.38 100.33 0)
-      (effects (font (size 1.27 1.27)) hide)
-    )
-    (pin "1")
-    (instances
-      (project "lab02"
-        (path "/352d7abe-fc72-4473-8b68-62eecf44f496/4087662f-8023-43e4-a97d-75c33092c189"
-          (reference "#PWR019") (unit 1)
         )
       )
@@
       (effects (font (size 1.27 1.27)) (justify left))
     )
-    (property "Footprint" "" (at 131.7752 111.76 0)
+    (property "Footprint" "Capacitor_SMD:C_0603_1608Metric" (at 131.7752 111.76 0)
       (effects (font (size 1.27 1.27)) hide)
     )
@@
         )
       )
-    )
-  )
-  (symbol (lib_id "power:+4V") (at 110.49 100.33 0) (unit 1)
-    (in_bom yes) (on_board yes) (dnp no) (fields_autoplaced)
-    (property "Reference" "#PWR015" (at 110.49 104.14 0)
-      (effects (font (size 1.27 1.27)) hide)
-    )
-    (property "Value" "+4V" (at 110.49 95.25 0)
-      (effects (font (size 1.27 1.27)))
-    )
-    (property "Footprint" "" (at 110.49 100.33 0)
-      (effects (font (size 1.27 1.27)) hide)
-    )
-    (property "Datasheet" "" (at 110.49 100.33 0)
-      (effects (font (size 1.27 1.27)) hide)
-    )
-    (pin "1")
-    (instances
-      (project "lab02"
-        (path "/352d7abe-fc72-4473-8b68-62eecf44f496/4087662f-8023-43e4-a97d-75c33092c189"
-          (reference "#PWR015") (unit 1)
-        )
-      )

Commit message: v5
Parts:
- J1: footprint (none) -> Connector_JST:JST_EH_S2B-EH_1x02_P2.50mm_Horizontal
Changed lines of the file:
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@@
       (effects (font (size 1.27 1.27)))
     )
-    (property "Footprint" "" (at 107.95 100.33 0)
+    (property "Footprint" "Connector_JST:JST_EH_S2B-EH_1x02_P2.50mm_Horizontal" (at 107.95 100.33 0)
       (effects (font (size 1.27 1.27)) hide)
     )

Commit message: v6
Parts:
- J1: Digikey PN (none) -> 455-S2B-EH-ND; MPN (none) -> S2B-EH
- U5: Digikey PN (none) -> AP2112K-3.3TRG1DICT-ND; MPN (none) -> AP2112K-3.3TRG1
Changed lines of the file:
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@@
+      (effects (font (size 1.27 1.27)) hide)
+    )
+    (property "Digikey PN" "AP2112K-3.3TRG1DICT-ND" (at 148.59 102.87 0)
+      (effects (font (size 1.27 1.27)) hide)
+    )
+    (property "MPN" "AP2112K-3.3TRG1" (at 148.59 102.87 0)
       (effects (font (size 1.27 1.27)) hide)
     )
@@
       (effects (font (size 1.27 1.27)) hide)
     )
-    (property "Datasheet" "~" (at 107.95 100.33 0)
+    (property "Datasheet" "https://www.jst-mfg.com/product/pdf/eng/eEH.pdf" (at 107.95 100.33 0)
       (effects (font (size 1.27 1.27)) hide)
     )
+    (property "Digikey PN" "455-S2B-EH-ND" (at 107.95 100.33 0)
+      (effects (font (size 1.27 1.27)) hide)
+    )
+    (property "MPN" "S2B-EH" (at 107.95 100.33 0)
+      (effects (font (size 1.27 1.27)) hide)
+    )

Commit message: pcb layout v0
Parts:
- added D4, D7: SS34, Diode_SMD:D_SMC, symbol Device:D_Small
Connections:
- net VBAT: now also D7.2 (A); no longer C2.1, U5.1 (VIN), U5.3 (EN)
- new net: C2.1, D4.1 (K), D7.1 (K), U5.1 (VIN), U5.3 (EN)
- new net VUSB: D4.2 (A)
Other:
- moved on the sheet: J1
Changed lines of the file:
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@@
   (junction (at 130.81 100.33) (diameter 0) (color 0 0 0 0)
   )
-  (junction (at 121.92 100.33) (diameter 0) (color 0 0 0 0)
-  )
-  (wire (pts (xy 121.92 95.25) (xy 121.92 100.33))
-    (stroke (width 0) (type default))
+  (junction (at 127 100.33) (diameter 0) (color 0 0 0 0)
+  )
+  (junction (at 114.3 100.33) (diameter 0) (color 0 0 0 0)
   )
   (wire (pts (xy 130.81 104.14) (xy 130.81 100.33))
     (stroke (width 0) (type default))
   )
-  (wire (pts (xy 113.03 100.33) (xy 121.92 100.33))
+  (wire (pts (xy 127 100.33) (xy 130.81 100.33))
+    (stroke (width 0) (type default))
+  )
+  (wire (pts (xy 127 86.36) (xy 127 88.9))
     (stroke (width 0) (type default))
   )
@@
     (stroke (width 0) (type default))
   )
+  (wire (pts (xy 127 93.98) (xy 127 100.33))
+    (stroke (width 0) (type default))
+  )
+  (wire (pts (xy 114.3 100.33) (xy 118.11 100.33))
+    (stroke (width 0) (type default))
+  )
   (wire (pts (xy 135.89 100.33) (xy 140.97 100.33))
     (stroke (width 0) (type default))
@@
     (stroke (width 0) (type default))
   )
-  (wire (pts (xy 121.92 100.33) (xy 130.81 100.33))
-    (stroke (width 0) (type default))
-  )
-  (wire (pts (xy 113.03 102.87) (xy 119.38 102.87))
-    (stroke (width 0) (type default))
-  )
-  (hierarchical_label "VBAT" (shape input) (at 121.92 95.25 0) (fields_autoplaced)
+  (wire (pts (xy 123.19 100.33) (xy 127 100.33))
+    (stroke (width 0) (type default))
+  )
+  (wire (pts (xy 114.3 86.36) (xy 114.3 100.33))
+    (stroke (width 0) (type default))
+  )
+  (wire (pts (xy 109.22 102.87) (xy 119.38 102.87))
+    (stroke (width 0) (type default))
+  )
+  (wire (pts (xy 109.22 100.33) (xy 114.3 100.33))
+    (stroke (width 0) (type default))
+  )
+  (hierarchical_label "VBAT" (shape input) (at 114.3 86.36 0) (fields_autoplaced)
     (effects (font (size 1.27 1.27)) (justify left))
   )
+  (hierarchical_label "VUSB" (shape input) (at 127 86.36 0) (fields_autoplaced)
+    (effects (font (size 1.27 1.27)) (justify left))
+  )
   (symbol (lib_id "power:GND") (at 119.38 102.87 0) (unit 1)
     (in_bom yes) (on_board yes) (dnp no) (fields_autoplaced)
@@
         (path "/352d7abe-fc72-4473-8b68-62eecf44f496/4087662f-8023-43e4-a97d-75c33092c189"
           (reference "#PWR016") (unit 1)
+        )
+      )
+    )
+  )
+  (symbol (lib_id "Device:D_Small") (at 127 91.44 90) (unit 1)
+    (in_bom yes) (on_board yes) (dnp no) (fields_autoplaced)
+    (property "Reference" "D4" (at 129.54 90.17 90)
+      (effects (font (size 1.27 1.27)) (justify right))
+    )
+    (property "Value" "SS34" (at 129.54 92.71 90)
+      (effects (font (size 1.27 1.27)) (justify right))
+    )
+    (property "Footprint" "Diode_SMD:D_SMC" (at 127 91.44 90)
+      (effects (font (size 1.27 1.27)) hide)
+    )
+    (property "Datasheet" "~" (at 127 91.44 90)
+      (effects (font (size 1.27 1.27)) hide)
+    )
+    (property "Sim.Device" "D" (at 127 91.44 0)
+      (effects (font (size 1.27 1.27)) hide)
+    )
+    (property "Sim.Pins" "1=K 2=A" (at 127 91.44 0)
+      (effects (font (size 1.27 1.27)) hide)
+    )
+    (pin "1")
+    (pin "2")
+    (instances
+      (project "lab02"
+        (path "/352d7abe-fc72-4473-8b68-62eecf44f496/4087662f-8023-43e4-a97d-75c33092c189"
+          (reference "D4") (unit 1)
         )
       )
@@
     )
   )
-  (symbol (lib_id "Connector:Conn_01x02_Pin") (at 107.95 100.33 0) (unit 1)
-    (in_bom yes) (on_board yes) (dnp no) (fields_autoplaced)
-    (property "Reference" "J1" (at 108.585 95.25 0)
-      (effects (font (size 1.27 1.27)))
-    )
-    (property "Value" "Conn_01x02_Pin" (at 108.585 97.79 0)
-      (effects (font (size 1.27 1.27)))
-    )
-    (property "Footprint" "Connector_JST:JST_EH_S2B-EH_1x02_P2.50mm_Horizontal" (at 107.95 100.33 0)
-      (effects (font (size 1.27 1.27)) hide)
-    )
-    (property "Datasheet" "https://www.jst-mfg.com/product/pdf/eng/eEH.pdf" (at 107.95 100.33 0)
-      (effects (font (size 1.27 1.27)) hide)
-    )
-    (property "Digikey PN" "455-S2B-EH-ND" (at 107.95 100.33 0)
-      (effects (font (size 1.27 1.27)) hide)
-    )
-    (property "MPN" "S2B-EH" (at 107.95 100.33 0)
+  (symbol (lib_id "Connector:Conn_01x02_Pin") (at 104.14 100.33 0) (unit 1)
+    (in_bom yes) (on_board yes) (dnp no) (fields_autoplaced)
+    (property "Reference" "J1" (at 104.775 95.25 0)
+      (effects (font (size 1.27 1.27)))
+    )
+    (property "Value" "Conn_01x02_Pin" (at 104.775 97.79 0)
+      (effects (font (size 1.27 1.27)))
+    )
+    (property "Footprint" "Connector_JST:JST_EH_S2B-EH_1x02_P2.50mm_Horizontal" (at 104.14 100.33 0)
+      (effects (font (size 1.27 1.27)) hide)
+    )
+    (property "Datasheet" "https://www.jst-mfg.com/product/pdf/eng/eEH.pdf" (at 104.14 100.33 0)
+      (effects (font (size 1.27 1.27)) hide)
+    )
+    (property "Digikey PN" "455-S2B-EH-ND" (at 104.14 100.33 0)
+      (effects (font (size 1.27 1.27)) hide)
+    )
+    (property "MPN" "S2B-EH" (at 104.14 100.33 0)
       (effects (font (size 1.27 1.27)) hide)
     )
@@
         )
       )
+    )
+  )
+  (symbol (lib_id "Device:D_Small") (at 120.65 100.33 180) (unit 1)
+    (in_bom yes) (on_board yes) (dnp no) (fields_autoplaced)
+    (property "Reference" "D7" (at 120.65 93.98 0)
+      (effects (font (size 1.27 1.27)))
+    )
+    (property "Value" "SS34" (at 120.65 96.52 0)
+      (effects (font (size 1.27 1.27)))
+    )
+    (property "Footprint" "Diode_SMD:D_SMC" (at 120.65 100.33 90)
+      (effects (font (size 1.27 1.27)) hide)
+    )
+    (property "Datasheet" "~" (at 120.65 100.33 90)
+      (effects (font (size 1.27 1.27)) hide)
+    )
+    (property "Sim.Device" "D" (at 120.65 100.33 0)
+      (effects (font (size 1.27 1.27)) hide)
+    )
+    (property "Sim.Pins" "1=K 2=A" (at 120.65 100.33 0)
+      (effects (font (size 1.27 1.27)) hide)
+    )
+    (pin "1")
+    (pin "2")
+    (instances
+      (project "lab02"
+        (path "/352d7abe-fc72-4473-8b68-62eecf44f496/4087662f-8023-43e4-a97d-75c33092c189"
+          (reference "D7") (unit 1)
+        )
+      )

Commit message: v7 pcb
Parts:
- J1: footprint Connector_JST:JST_EH_S2B-EH_1x02_P2.50mm_Horizontal -> lab02_components:JST_B2B-XH-A; Digikey PN 455-S2B-EH-ND -> 455-B2B-XH-A-ND; MPN S2B-EH -> B2B-XH-A
Changed lines of the file:
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@@
       (effects (font (size 1.27 1.27)))
     )
-    (property "Footprint" "Connector_JST:JST_EH_S2B-EH_1x02_P2.50mm_Horizontal" (at 104.14 100.33 0)
+    (property "Footprint" "lab02_components:JST_B2B-XH-A" (at 104.14 100.33 0)
       (effects (font (size 1.27 1.27)) hide)
     )
-    (property "Datasheet" "https://www.jst-mfg.com/product/pdf/eng/eEH.pdf" (at 104.14 100.33 0)
+    (property "Datasheet" "https://www.jst-mfg.com/product/pdf/eng/eXH.pdf" (at 104.14 100.33 0)
       (effects (font (size 1.27 1.27)) hide)
     )
-    (property "Digikey PN" "455-S2B-EH-ND" (at 104.14 100.33 0)
+    (property "Digikey PN" "455-B2B-XH-A-ND" (at 104.14 100.33 0)
       (effects (font (size 1.27 1.27)) hide)
     )
-    (property "MPN" "S2B-EH" (at 104.14 100.33 0)
+    (property "MPN" "B2B-XH-A" (at 104.14 100.33 0)
       (effects (font (size 1.27 1.27)) hide)
     )
