File: lab02/voltage.kicad_sch (KiCad schematic)
At the start: 0 parts

Commit message: v1
Parts:
- added C1: 1nF, Capacitor_SMD:C_0603_1608Metric, symbol Device:C
- added D6: 51V, symbol Device:D_Zener
- added R10: 200k, symbol Device:R_Small
- added R11: 10k, symbol Device:R_Small
- added R8: 160R, symbol Device:R_Small
- added U4: OPA310 DBV, lab02_components:SOT-23-5-DBV_TEX, symbol Amplifier_Operational:OPA188xxDBV
Connections:
- new net: R10.2, R11.1, U4.3 (+)
- new net: R8.2, U4.1, U4.4 (-)
- new net +3.3V: U4.5 (V+)
- new net GND: C1.2, D6.2 (A), R11.2, U4.2 (V-)
- new net PGA_V: C1.1, R8.1
- new net P_V+: D6.1 (K), R10.1

Commit message: v2
Changed lines of the file:
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@@
     (stroke (width 0) (type default))
-  )
-  (global_label "P_V+" (shape input) (at 170.18 90.17 0) (fields_autoplaced)
-    (effects (font (size 1.27 1.27)) (justify left))
-    (property "Intersheetrefs" "${INTERSHEET_REFS}" (at 178.0638 90.17 0)
-      (effects (font (size 1.27 1.27)) (justify left) hide)
-    )
-  )
-  (global_label "P-" (shape input) (at 170.18 107.95 0) (fields_autoplaced)
-    (effects (font (size 1.27 1.27)) (justify left))
-    (property "Intersheetrefs" "${INTERSHEET_REFS}" (at 176.0076 107.95 0)
-      (effects (font (size 1.27 1.27)) (justify left) hide)
-    )
   )
   (hierarchical_label "PGA_V" (shape input) (at 92.71 96.52 180) (fields_autoplaced)
     (effects (font (size 1.27 1.27)) (justify right))
   )
+  (hierarchical_label "P_V+" (shape input) (at 170.18 90.17 0) (fields_autoplaced)
+    (effects (font (size 1.27 1.27)) (justify left))
+  )
+  (hierarchical_label "P-" (shape input) (at 170.18 107.95 0) (fields_autoplaced)
+    (effects (font (size 1.27 1.27)) (justify left))
+  )
   (symbol (lib_id "Device:D_Zener") (at 162.56 99.06 270) (unit 1)

Commit message: v3
Parts:
- U4: value OPA310 DBV -> OPA310IDBVR; footprint lab02_components:SOT-23-5-DBV_TEX -> lab02_components:OPA310IDBVR; Digikey PN (none) -> 296-OPA310IDBVRCT-ND; MPN (none) -> OPA310IDBVR
Changed lines of the file:
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@@
       (effects (font (size 1.27 1.27)) (justify right))
     )
-    (property "Value" "OPA310 DBV" (at 133.6959 88.9 0)
+    (property "Value" "OPA310IDBVR" (at 133.6959 88.9 0)
       (effects (font (size 1.27 1.27)) (justify right))
     )
-    (property "Footprint" "lab02_components:SOT-23-5-DBV_TEX" (at 130.81 96.52 0)
+    (property "Footprint" "lab02_components:OPA310IDBVR" (at 130.81 96.52 0)
       (effects (font (size 1.27 1.27)) hide)
     )
-    (property "Datasheet" "https://www.ti.com/lit/ds/symlink/opa310.pdf?ts=1705006057026&ref_url=https%253A%252F%252Fwww.ti.com%252Fproduct%252FOPA310" (at 130.81 101.6 0)
+    (property "Datasheet" "https://www.ti.com/lit/ds/symlink/opa310.pdf" (at 130.81 101.6 0)
       (effects (font (size 1.27 1.27)) hide)
     )
+    (property "Digikey PN" "296-OPA310IDBVRCT-ND" (at 130.81 96.52 0)
+      (effects (font (size 1.27 1.27)) hide)
+    )
+    (property "MPN" "OPA310IDBVR" (at 130.81 96.52 0)
+      (effects (font (size 1.27 1.27)) hide)
+    )

Commit message: v4
Parts:
- R10: value 200k -> 200K; footprint (none) -> Resistor_SMD:R_0603_1608Metric
- R11: value 10k -> 10K; footprint (none) -> Resistor_SMD:R_0603_1608Metric
- R8: footprint (none) -> Resistor_SMD:R_0603_1608Metric
Changed lines of the file:
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@@
       (effects (font (size 1.27 1.27)) (justify left))
     )
-    (property "Value" "10k" (at 153.67 106.68 0)
-      (effects (font (size 1.27 1.27)) (justify left))
-    )
-    (property "Footprint" "" (at 151.13 105.41 0)
+    (property "Value" "10K" (at 153.67 106.68 0)
+      (effects (font (size 1.27 1.27)) (justify left))
+    )
+    (property "Footprint" "Resistor_SMD:R_0603_1608Metric" (at 151.13 105.41 0)
       (effects (font (size 1.27 1.27)) hide)
     )
@@
       (effects (font (size 1.27 1.27)) (justify left))
     )
-    (property "Value" "200k" (at 153.67 93.98 0)
-      (effects (font (size 1.27 1.27)) (justify left))
-    )
-    (property "Footprint" "" (at 151.13 92.71 0)
+    (property "Value" "200K" (at 153.67 93.98 0)
+      (effects (font (size 1.27 1.27)) (justify left))
+    )
+    (property "Footprint" "Resistor_SMD:R_0603_1608Metric" (at 151.13 92.71 0)
       (effects (font (size 1.27 1.27)) hide)
     )
@@
       (effects (font (size 1.27 1.27)))
     )
-    (property "Footprint" "" (at 113.03 96.52 0)
-      (effects (font (size 1.27 1.27)) hide)
-    )
+    (property "Footprint" "Resistor_SMD:R_0603_1608Metric" (at 113.03 96.52 0)
+      (effects (font (size 1.27 1.27)) hide)
+    )

Commit message: v7
Parts:
- added C8: 100nF, Capacitor_SMD:C_0603_1608Metric, symbol Device:C
- D6: footprint (none) -> lab02_components:BZT52C51-7-F; Digikey PN (none) -> BZT52C51-FDICT-ND; MPN (none) -> BZT52C51-7-F
Connections:
- net +3.3V: now also C8.1
- net GND: now also C8.2
Changed lines of the file:
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@@
   (junction (at 151.13 99.06) (diameter 0) (color 0 0 0 0)
   )
+  (junction (at 130.81 104.14) (diameter 0) (color 0 0 0 0)
+  )
   (junction (at 120.65 96.52) (diameter 0) (color 0 0 0 0)
   )
@@
     (stroke (width 0) (type default))
   )
+  (wire (pts (xy 130.81 104.14) (xy 133.35 104.14))
+    (stroke (width 0) (type default))
+  )
   (wire (pts (xy 138.43 93.98) (xy 140.97 93.98))
     (stroke (width 0) (type default))
@@
     (stroke (width 0) (type default))
   )
-  (wire (pts (xy 129.54 104.14) (xy 133.35 104.14))
+  (wire (pts (xy 129.54 104.14) (xy 130.81 104.14))
     (stroke (width 0) (type default))
   )
@@
       (effects (font (size 1.27 1.27)) (justify left))
     )
-    (property "Footprint" "" (at 162.56 99.06 0)
-      (effects (font (size 1.27 1.27)) hide)
-    )
-    (property "Datasheet" "~" (at 162.56 99.06 0)
+    (property "Footprint" "lab02_components:BZT52C51-7-F" (at 162.56 99.06 0)
+      (effects (font (size 1.27 1.27)) hide)
+    )
+    (property "Datasheet" "https://www.diodes.com/assets/Datasheets/ds18004.pdf" (at 162.56 99.06 0)
+      (effects (font (size 1.27 1.27)) hide)
+    )
+    (property "Digikey PN" "BZT52C51-FDICT-ND" (at 162.56 99.06 0)
+      (effects (font (size 1.27 1.27)) hide)
+    )
+    (property "MPN" "BZT52C51-7-F" (at 162.56 99.06 0)
       (effects (font (size 1.27 1.27)) hide)
     )
@@
     )
   )
+  (symbol (lib_id "power:GND") (at 130.81 111.76 0) (unit 1)
+    (in_bom yes) (on_board yes) (dnp no) (fields_autoplaced)
+    (property "Reference" "#PWR043" (at 130.81 118.11 0)
+      (effects (font (size 1.27 1.27)) hide)
+    )
+    (property "Value" "GND" (at 130.81 116.84 0)
+      (effects (font (size 1.27 1.27)))
+    )
+    (property "Footprint" "" (at 130.81 111.76 0)
+      (effects (font (size 1.27 1.27)) hide)
+    )
+    (property "Datasheet" "" (at 130.81 111.76 0)
+      (effects (font (size 1.27 1.27)) hide)
+    )
+    (pin "1")
+    (instances
+      (project "lab02"
+        (path "/352d7abe-fc72-4473-8b68-62eecf44f496/cc5f35a2-1c02-4b49-920c-b58faab8810e"
+          (reference "#PWR043") (unit 1)
+        )
+      )
+    )
+  )
   (symbol (lib_id "Amplifier_Operational:OPA188xxDBV") (at 130.81 96.52 180) (unit 1)
     (in_bom yes) (on_board yes) (dnp no) (fields_autoplaced)
@@
         )
       )
+    )
+  )
+  (symbol (lib_id "Device:C") (at 130.81 107.95 0) (unit 1)
+    (in_bom yes) (on_board yes) (dnp no)
+    (property "Reference" "C8" (at 124.46 106.68 0)
+      (effects (font (size 1.27 1.27)) (justify left))
+    )
+    (property "Value" "100nF" (at 121.92 109.22 0)
+      (effects (font (size 1.27 1.27)) (justify left))
+    )
+    (property "Footprint" "Capacitor_SMD:C_0603_1608Metric" (at 131.7752 111.76 0)
+      (effects (font (size 1.27 1.27)) hide)
+    )
+    (property "Datasheet" "~" (at 130.81 107.95 0)
+      (effects (font (size 1.27 1.27)) hide)
+    )
+    (pin "2")
+    (pin "1")
+    (instances
+      (project "lab02"
+        (path "/352d7abe-fc72-4473-8b68-62eecf44f496/cc5f35a2-1c02-4b49-920c-b58faab8810e"
+          (reference "C8") (unit 1)
+        )
+      )

Commit message: v7 pcb
Parts:
- added D8: 51V, lab02_components:BZT52C51-7-F, symbol Device:D_Zener
Connections:
- net GND: now also D8.1 (K); no longer D6.2 (A)
- new net: D6.2 (A), D8.2 (A)
Other:
- moved on the sheet: D6
Changed lines of the file:
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@@
     (stroke (width 0) (type default))
   )
-  (wire (pts (xy 162.56 90.17) (xy 162.56 95.25))
+  (wire (pts (xy 162.56 90.17) (xy 162.56 91.44))
     (stroke (width 0) (type default))
   )
@@
     (stroke (width 0) (type default))
   )
-  (wire (pts (xy 162.56 102.87) (xy 162.56 107.95))
-    (stroke (width 0) (type default))
-  )
   (wire (pts (xy 129.54 104.14) (xy 130.81 104.14))
+    (stroke (width 0) (type default))
+  )
+  (wire (pts (xy 162.56 106.68) (xy 162.56 107.95))
     (stroke (width 0) (type default))
   )
@@
     (effects (font (size 1.27 1.27)) (justify left))
   )
-  (symbol (lib_id "Device:D_Zener") (at 162.56 99.06 270) (unit 1)
-    (in_bom yes) (on_board yes) (dnp no) (fields_autoplaced)
-    (property "Reference" "D6" (at 165.1 97.79 90)
-      (effects (font (size 1.27 1.27)) (justify left))
-    )
-    (property "Value" "51V" (at 165.1 100.33 90)
-      (effects (font (size 1.27 1.27)) (justify left))
-    )
-    (property "Footprint" "lab02_components:BZT52C51-7-F" (at 162.56 99.06 0)
-      (effects (font (size 1.27 1.27)) hide)
-    )
-    (property "Datasheet" "https://www.diodes.com/assets/Datasheets/ds18004.pdf" (at 162.56 99.06 0)
-      (effects (font (size 1.27 1.27)) hide)
-    )
-    (property "Digikey PN" "BZT52C51-FDICT-ND" (at 162.56 99.06 0)
-      (effects (font (size 1.27 1.27)) hide)
-    )
-    (property "MPN" "BZT52C51-7-F" (at 162.56 99.06 0)
+  (symbol (lib_id "Device:D_Zener") (at 162.56 95.25 270) (unit 1)
+    (in_bom yes) (on_board yes) (dnp no) (fields_autoplaced)
+    (property "Reference" "D6" (at 165.1 93.98 90)
+      (effects (font (size 1.27 1.27)) (justify left))
+    )
+    (property "Value" "51V" (at 165.1 96.52 90)
+      (effects (font (size 1.27 1.27)) (justify left))
+    )
+    (property "Footprint" "lab02_components:BZT52C51-7-F" (at 162.56 95.25 0)
+      (effects (font (size 1.27 1.27)) hide)
+    )
+    (property "Datasheet" "https://www.diodes.com/assets/Datasheets/ds18004.pdf" (at 162.56 95.25 0)
+      (effects (font (size 1.27 1.27)) hide)
+    )
+    (property "Digikey PN" "BZT52C51-FDICT-ND" (at 162.56 95.25 0)
+      (effects (font (size 1.27 1.27)) hide)
+    )
+    (property "MPN" "BZT52C51-7-F" (at 162.56 95.25 0)
       (effects (font (size 1.27 1.27)) hide)
     )
@@
         )
       )
+    )
+  )
+  (symbol (lib_id "Device:D_Zener") (at 162.56 102.87 90) (unit 1)
+    (in_bom yes) (on_board yes) (dnp no) (fields_autoplaced)
+    (property "Reference" "D8" (at 165.1 101.6 90)
+      (effects (font (size 1.27 1.27)) (justify right))
+    )
+    (property "Value" "51V" (at 165.1 104.14 90)
+      (effects (font (size 1.27 1.27)) (justify right))
+    )
+    (property "Footprint" "lab02_components:BZT52C51-7-F" (at 162.56 102.87 0)
+      (effects (font (size 1.27 1.27)) hide)
+    )
+    (property "Datasheet" "https://www.diodes.com/assets/Datasheets/ds18004.pdf" (at 162.56 102.87 0)
+      (effects (font (size 1.27 1.27)) hide)
+    )
+    (property "Digikey PN" "BZT52C51-FDICT-ND" (at 162.56 102.87 0)
+      (effects (font (size 1.27 1.27)) hide)
+    )
+    (property "MPN" "BZT52C51-7-F" (at 162.56 102.87 0)
+      (effects (font (size 1.27 1.27)) hide)
+    )
+    (pin "2")
+    (pin "1")
+    (instances
+      (project "lab02"
+        (path "/352d7abe-fc72-4473-8b68-62eecf44f496/cc5f35a2-1c02-4b49-920c-b58faab8810e"
+          (reference "D8") (unit 1)
+        )
+      )
