File: lab02/lab02.kicad_pcb (KiCad board)
At the start: 4 copper layers, 0 parts

Commit message: pcb layout v0
Parts:
- added C1: 1nF, Capacitor_SMD:C_0603_1608Metric, F.Cu at (145.0, 135.0)
- added C10: 100nF, Capacitor_SMD:C_0603_1608Metric, F.Cu at (105.0, 140.0)
- added C2: 1uF, Capacitor_SMD:C_0603_1608Metric, F.Cu at (144.2, 120.0)
- added C3: 1uF, Capacitor_SMD:C_0603_1608Metric, F.Cu at (143.3, 127.5)
- added C4: 0.1uF, Capacitor_SMD:C_0603_1608Metric, F.Cu at (128.1, 75.3)
- added C5: 0.1uF, Capacitor_SMD:C_0603_1608Metric, F.Cu at (128.1, 77.9)
- added C6: 0.1uF, Capacitor_SMD:C_0603_1608Metric, F.Cu at (128.1, 80.4)
- added C7: 0.1uF, Capacitor_SMD:C_0603_1608Metric, F.Cu at (114.7, 132.3)
- added C8: 100nF, Capacitor_SMD:C_0603_1608Metric, F.Cu at (140.0, 144.2)
- added C9: 1uF, Capacitor_SMD:C_0603_1608Metric, F.Cu at (128.1, 82.9)
- added D1: 3.3V, lab02_components:MMSZ4684T1G, F.Cu at (111.7, 140.0)
- added D2: GREEN LED, LED_SMD:LED_0603_1608Metric_Pad1.05x0.95mm_HandSolder, F.Cu at (134.3, 94.9)
- added D3: GREEN LED, LED_SMD:LED_0603_1608Metric_Pad1.05x0.95mm_HandSolder, F.Cu at (131.7, 94.9)
- added D4: SS34, Diode_SMD:D_SMC, F.Cu at (135.9, 123.1)
- added D5: GREEN LED, LED_SMD:LED_0603_1608Metric_Pad1.05x0.95mm_HandSolder, F.Cu at (129.1, 94.9)
- added D6: 51V, lab02_components:BZT52C51-7-F, F.Cu at (145.0, 140.0)
- added D7: SS34, Diode_SMD:D_SMC, F.Cu at (135.9, 130.9)
- added F1: 10A Fuse, lab02_components:FUSE_31.8221_SCH, F.Cu at (115.9, 124.8)
- added J1: Conn_01x02_Pin, Connector_JST:JST_EH_S2B-EH_1x02_P2.50mm_Horizontal, F.Cu at (128.4, 140.0)
- added J2: Conn_01x04_Pin, lab02_components:PPTC041LFBN-RC, F.Cu at (142.2, 95.4)
- added J3: USB_C_Receptacle_USB2.0_14P, lab02_components:USB4085-GF-A, F.Cu at (150.9, 78.3)
- added J4: FCR7350R, lab02_components:CONN1_FCR7350R_CLF, F.Cu at (144.8, 66.4)
- added J5: FCR7350R, lab02_components:CONN1_FCR7350R_CLF, F.Cu at (130.1, 66.4)
- added J6: FCR7350B, lab02_components:CONN1_FCR7350R_CLF, F.Cu at (115.4, 66.4)
- added NT1: NetTie_2, NetTie:NetTie-2_SMD_Pad0.5mm, F.Cu at (135.5, 95.8)
- added R1: 100K, Resistor_SMD:R_0603_1608Metric, F.Cu at (116.0, 143.0)
- added R10: 200K, Resistor_SMD:R_0603_1608Metric, F.Cu at (145.0, 144.5)
- added R11: 10K, Resistor_SMD:R_0603_1608Metric, F.Cu at (150.0, 145.0)
- added R12: 10K, Resistor_SMD:R_0603_1608Metric, F.Cu at (132.1, 77.9)
- added R13: 2K, Resistor_SMD:R_0603_1608Metric, F.Cu at (132.1, 80.4)
- added R14: 10K, Resistor_SMD:R_0603_1608Metric, F.Cu at (132.1, 82.9)
- added R15: 2K, Resistor_SMD:R_0603_1608Metric, F.Cu at (132.1, 85.4)
- added R16: 2K, Resistor_SMD:R_0603_1608Metric, F.Cu at (132.1, 87.9)
- added R17: 442K, Resistor_SMD:R_0603_1608Metric, F.Cu at (132.1, 90.4)
- added R18: 160K, Resistor_SMD:R_0603_1608Metric, F.Cu at (136.1, 75.3)
- added R2: 2K, Resistor_SMD:R_0603_1608Metric, F.Cu at (128.1, 85.4)
- added R20: 5.1K, Resistor_SMD:R_0603_1608Metric, F.Cu at (136.1, 77.9)
- added R21: 5.1K, Resistor_SMD:R_0603_1608Metric, F.Cu at (136.1, 80.4)
- added R22: 10K, Resistor_SMD:R_0603_1608Metric, F.Cu at (136.1, 82.9)
- added R23: 5.1K, Resistor_SMD:R_0603_1608Metric, F.Cu at (136.1, 85.4)
- added R3: 10K, Resistor_SMD:R_0603_1608Metric, F.Cu at (128.1, 87.9)
- added R4: 2K, Resistor_SMD:R_0603_1608Metric, F.Cu at (128.1, 90.4)
- added R5: 100R, Resistor_SMD:R_0603_1608Metric, F.Cu at (132.1, 75.3)
- added R6: 1mR, lab02_components:CSNL1206FT1L00, F.Cu at (119.4, 132.8)
- added R7: 340R, Resistor_SMD:R_0603_1608Metric, F.Cu at (114.7, 134.8)
- added R8: 160R, Resistor_SMD:R_0603_1608Metric, F.Cu at (150.0, 134.2)
- added R9: 0R, Resistor_SMD:R_0603_1608Metric, F.Cu at (114.7, 137.3)
- added SW1: SW_SPST, lab02_components:SWITCH_FSMSM_TYC, F.Cu at (132.7, 105.4)
- added SW2: SW_SPST, lab02_components:SWITCH_FSMSM_TYC, F.Cu at (126.8, 105.4)
- added SW3: SW_SPST, lab02_components:SWITCH_FSMSM_TYC, F.Cu at (120.9, 105.4)
- added SW4: SW_SPST, lab02_components:SWITCH_FSMSM_TYC, F.Cu at (105.9, 105.4)
- added SW5: SW_SPST, lab02_components:SWITCH_FSMSM_TYC, F.Cu at (105.9, 111.3)
- added U1: OPA310IDBVR, lab02_components:OPA310IDBVR, F.Cu at (111.3, 144.2)
- added U2: INA823, Package_SO:SOIC-8_3.9x4.9mm_P1.27mm, F.Cu at (108.4, 134.2)
- added U3: PGA116AIPW, lab02_components:PGA116AIPWR, F.Cu at (143.9, 89.2)
- added U4: OPA310IDBVR, lab02_components:OPA310IDBVR, F.Cu at (150.0, 139.8)
- added U5: AP2112K-3.3, Package_TO_SOT_SMD:SOT-23-5, F.Cu at (148.9, 121.5)
- added U7: ESP32-S3-WROOM-1-N4, lab02_components:ESP32-S3-WROOM-1-N4, F.Cu at (115.8, 86.7)
Routing:
- net Net-(D4-K): track 0.00 -> 28.1 mm
- net /vbat: track 0.00 -> 19.2 mm
- net /p+_v-r: track 0.00 -> 9.34 mm
- net Net-(U4--): track 0.00 -> 7.85 mm
- net Net-(U4-+): track 0.00 -> 7.71 mm
- net /pga_v: track 0.00 -> 3.74 mm
- net /pga_r: track 0.00 -> 3.52 mm
Other:
- board outline added: 60 x 100 mm

Commit message: pcb layout v1
Parts:
- moved C10 12.7 mm to (116.6, 145.2)
- moved C7 12.1 mm to (105.3, 140.0), turned to 180 degrees
- moved D1 11.6 mm to (123.3, 140.0)
- moved R1 11.6 mm to (127.6, 143.0)
- moved U1 11.6 mm to (122.9, 144.2)
- moved R9 9.58 mm to (105.3, 135.0), turned to -90 degrees
- moved J1 6.60 mm to (135.0, 140.0)
- moved R7 5.23 mm to (115.0, 140.0), turned to 180 degrees
- moved U2 4.28 mm to (112.5, 135.6), turned to 180 degrees
- moved R6 2.30 mm to (120.0, 135.0), turned to -90 degrees
- moved J4 0.36 mm to (144.8, 66.0)
- moved J5 0.36 mm to (130.1, 66.0)
- moved J6 0.36 mm to (115.4, 66.0)
Routing:
- net Net-(U2-+IN): track 0.00 -> 16.2 mm
- net /vbat: track 19.2 -> 11.9 mm
- net Net-(R7-Pad2): track 0.00 -> 5.19 mm
- net Net-(U2-REF): track 0.00 -> 4.84 mm
- net Net-(R7-Pad1): track 0.00 -> 2.82 mm

Commit message: v3
Parts:
- moved J3 48.4 mm to (105.6, 95.4), turned to -90 degrees
- moved R13 31.2 mm to (122.4, 110.0), turned to -90 degrees
- moved R2 28.9 mm to (143.2, 110.0), turned to -90 degrees
- moved R12 28.8 mm to (122.4, 105.0)
- moved R20 28.0 mm to (114.0, 95.0)
- moved R21 28.0 mm to (114.0, 97.5)
- moved SW5 26.3 mm to (105.0, 85.0)
- moved SW4 25.4 mm to (105.0, 80.0)
- moved R3 22.8 mm to (143.2, 105.0)
- moved D2 22.4 mm to (144.0, 115.0), turned to 0 degrees
- moved R22 22.3 mm to (115.0, 90.0), turned to -90 degrees
- moved R14 22.2 mm to (133.2, 105.0)
- moved D5 21.0 mm to (123.2, 115.0), turned to 0 degrees
- moved D3 20.3 mm to (134.0, 115.0), turned to 0 degrees
- moved R4 20.2 mm to (133.2, 110.0), turned to -90 degrees
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Connections:
- R12 pad 1: Net-(U7-IO8) -> Net-(U7-IO9)
- R13 pad 1: Net-(U7-IO8) -> Net-(U7-IO9)
- R14 pad 1: Net-(U7-IO12) -> Net-(U7-IO10)
- R2 pad 1: Net-(U7-IO10) -> Net-(U7-IO12)
- R3 pad 1: Net-(U7-IO10) -> Net-(U7-IO12)
- R4 pad 1: Net-(U7-IO12) -> Net-(U7-IO10)
- SW1 pad 1: Net-(U7-IO10) -> Net-(U7-IO12)
- SW2 pad 1: Net-(U7-IO12) -> Net-(U7-IO10)
- SW3 pad 1: Net-(U7-IO8) -> Net-(U7-IO9)
- U7 pad 12: Net-(U7-IO8) -> unconnected-(U7-IO8-Pad12)
- U7 pad 17: unconnected-(U7-IO9-Pad17) -> Net-(U7-IO9)
Routing:
- net Net-(D4-K): track 28.1 -> 15.9 mm
- net /vbat: track 11.9 -> 0.00 mm
- net Net-(U2-+IN): track 16.2 -> 12.6 mm

Commit message: v7 pcb
Parts:
- removed R17: 442K, Resistor_SMD:R_0603_1608Metric
- removed R18: 160K, Resistor_SMD:R_0603_1608Metric
- added D8: 51V, lab02_components:BZT52C51-7-F, F.Cu at (161.1, 92.5)
- J1: footprint Connector_JST:JST_EH_S2B-EH_1x02_P2.50mm_Horizontal -> lab02_components:JST_B2B-XH-A
- moved C10 74.9 mm to (160.9, 84.8), turned to -90 degrees
- moved R1 71.3 mm to (161.0, 80.0)
- moved U1 67.8 mm to (156.0, 85.0), turned to 0 degrees
- moved D1 67.1 mm to (153.3, 80.0)
- moved R10 60.1 mm to (172.0, 92.4), turned to -90 degrees
- moved R9 58.1 mm to (109.0, 77.0), turned to 0 degrees
- moved SW5 57.0 mm to (150.0, 120.0), turned to -90 degrees
- moved R6 55.6 mm to (116.6, 79.5), turned to 180 degrees
- moved R7 54.4 mm to (111.0, 85.7)
- moved U2 54.4 mm to (108.5, 81.4)
- moved C7 54.0 mm to (103.6, 86.1), turned to -90 degrees
- moved R11 53.8 mm to (172.0, 97.4)
- moved D6 53.8 mm to (167.0, 92.5), turned to -90 degrees
- moved R22 52.6 mm to (155.0, 124.2), turned to 90 degrees
- moved C8 51.3 mm to (161.0, 99.0), turned to -90 degrees
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Connections:
- D6 pad 2: GND -> Net-(D6-A)
- R12 pad 1: Net-(U7-IO9) -> Net-(U7-IO3)
- R2 pad 1: Net-(U7-IO12) -> Net-(U7-IO13)
- R4 pad 1: Net-(U7-IO10) -> Net-(U7-IO11)
- R5 pad 1: Net-(U7-IO5) -> /pga-v_o-adc
- R5 pad 2: /pga-v_o-adc -> Net-(U7-IO2)
- SW3 pad 1: Net-(U7-IO9) -> Net-(U7-IO3)
- U7 pad 15: unconnected-(U7-IO3-Pad15) -> Net-(U7-IO3)
- U7 pad 19: unconnected-(U7-IO11-Pad19) -> Net-(U7-IO11)
- U7 pad 21: /SDA -> Net-(U7-IO13)
- U7 pad 22: /SCL -> unconnected-(U7-IO14-Pad22)
- U7 pad 24: unconnected-(U7-IO47-Pad24) -> /SCL
- U7 pad 25: unconnected-(U7-IO48-Pad25) -> /SDA
- U7 pad 29: /SDO_ESP-SDI_PGA -> /SDI_ESP-SDO_PGA
- U7 pad 30: /SDI_ESP-SDO_PGA -> /SDO_ESP-SDI_PGA
- U7 pad 38: unconnected-(U7-IO2-Pad38) -> Net-(U7-IO2)
- U7 pad 39: Net-(U7-IO1) -> unconnected-(U7-IO1-Pad39)
- U7 pad 5: Net-(U7-IO5) -> unconnected-(U7-IO5-Pad5)
Routing:
- net /pga_i: track 0.00 -> 73.3 mm
- net /vusb: track 0.00 -> 58.7 mm
- net /p+_v-r: track 9.34 -> 52.0 mm
- net +3.3V: track 0.00 -> 29.3 mm
- net /pga_r: track 3.52 -> 30.9 mm
- net Net-(U7-IO9): track 0.00 -> 24.4 mm
- net GND: track 0.00 -> 24.0 mm
- net Net-(U7-IO3): track 0.00 -> 22.5 mm
- net Net-(U7-IO13): track 0.00 -> 22.1 mm
- net Net-(U7-IO11): track 0.00 -> 21.6 mm
- net /USB_P: track 0.00 -> 20.3 mm, vias 0 -> 2
- net /USB_N: track 0.00 -> 19.8 mm
- net Net-(U7-IO12): track 0.00 -> 19.6 mm
- net Net-(U7-IO10): track 0.00 -> 19.6 mm
- net /reset: track 0.00 -> 19.4 mm
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- added copper zone on F.Cu, net Net-(U2-+IN)
Other:
- board size 60 x 100 mm -> 75 x 100 mm
- copper layers 4 -> 2
- board text added: "3V3"
- board text added: "A"
- board text added: "COM"
- board text added: "CURRENT MEASUREMENT"
- board text added: "ESP boot"
- board text added: "ESP reset"
- board text added: "OLED screen"
- board text added: "PGA"
- board text added: "POWER SUPPLY"
- board text added: "RESISTANCE MEASUREMENT"
- board text added: "USB_C"
- board text added: "VOLTAGE MEASUREMENT"
- board text added: "VΩ"
- board text added: "current"
- board text added: "resistance"
- board text added: "voltage"

Commit message: v8
Parts:
- added H1: MountingHole, MountingHole:MountingHole_2.5mm, F.Cu at (169.9, 56.4)
- added H2: MountingHole, MountingHole:MountingHole_2.5mm, F.Cu at (106.9, 56.4)
- added H3: MountingHole, MountingHole:MountingHole_2.5mm, F.Cu at (106.9, 144.3)
- added H4: MountingHole, MountingHole:MountingHole_2.5mm, F.Cu at (169.9, 144.4)
- J3: footprint lab02_components:USB4085-GF-A -> Connector_USB:USB_C_Receptacle_GCT_USB4085
- U7: footprint lab02_components:ESP32-S3-WROOM-1-N4 -> RF_Module:ESP32-S3-WROOM-1
- moved J3 5.27 mm to (106.9, 107.8)
- moved R15 1.00 mm to (139.0, 124.1)
- moved R16 0.60 mm to (139.7, 119.5), turned to 0 degrees
Routing:
- net +3.3V: track 29.3 -> 231.1 mm
- net GND: track 24.0 -> 68.1 mm, vias 0 -> 31
- net /vusb: track 58.7 -> 63.8 mm
- net /SDA: track 10.0 -> 11.5 mm, vias 0 -> 1
- net Net-(D4-K): track 30.2 -> 31.2 mm
- net /USB_P: track 20.3 -> 19.3 mm
- net Net-(U7-IO3): track 22.5 -> 21.9 mm
- net /SCL: track 13.9 -> 14.5 mm, vias 0 -> 1
- net /reset: track 19.4 -> 20.0 mm
- added copper zone on B.Cu, net GND
Other:
- board size 75 x 100 mm -> 75.3 x 100 mm

Commit message: v9
Parts:
- added H5: logo1, lab02_components:EdgertonLogo, F.Cu at (148.7, 142.3)
- added H6: logo2, lab02_components:EECSLogo, F.Cu at (142.8, 91.6)
- added H7: logo1, lab02_components:MechE, F.Cu at (167.2, 73.3)
